File: electronics/power-hub/controller.kicad_sch (KiCad schematic)
At the start: 56 parts, among them J6 USB, SW1 RESET, SW2 BOOT, U2 LMR51635YDDCR, U3 AP2112K-3.3TRG1, U4 ESP32-S3-MINI-1-N8, U5 USBLC6-2SC6, U6 TJA1462AT

Commit message: Power hub: CH224A PD sink instead of the AP33772S, no input switch
The AP33772S has no LCSC stock (Global Sourcing only).  The WCH CH224A
(C42459160, in stock) takes its place in the one-resistor mode: CFG1 6.8k
asks for 9 V at plug-in and turns I2C on, so the controller asks for 28 V
EPR (else 20 V) over I2C.  PG (open drain) keeps the PD_INT net: IO39 and
the front PD LED.  Its supply (VHV and VBUS tied) runs through 56 ohm +
1 uF: the pins are rated 32 V.

No input switch: VBUS is VRACK, and the eFuses (off until enabled, UV 15 V,
reverse blocking) do the switching.  Out: the IRF7842 pair, the 5 mohm
shunt, the NTC and their passives.  Re-routed: ERC 0, DRC 0, parity 0.
37 -> 33 part types; the hub order about $185 (BOM adjustments).  Docs:
power.md, electronics.md, sourcing.md.

Co-Authored-By: Claude Opus 5.5 <noreply@anthropic.com>
Parts:
- removed TP8: PD_VCC, TestPoint:TestPoint_Pad_D1.5mm, symbol Connector:TestPoint
Connections:
- net PD_VCC is gone; now on net VRACK: C104.1, C105.1, C106.1, R205.1, U2.3 (VIN)
Other:
- moved on the sheet: C116, C117, C118, C119, C120, D9, H1, H2, H3, H4, J6, R212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

Commit message: PCBA review: hub and node fixes before the order
On main's CH224A hub and the bay node v0.5.

Power hub:
- CPL: the side LEDs (C598310, C4555382) +0.825 mm, their polarity
  proven from JLC's own footprints (and C495809 at 270 deg in the table,
  for the IRF7842 the AP33772S hub had).
- Rows: SHDN pull-downs 10k, so rows stay off without firmware (100k
  gave 1 V at the pin's 10 uA); a B5819W at each row output for the
  cable's kick; the red FAULT LEDs fed from their ROW_EN, so a row that
  is simply off shows no fault.
- In2's VRACK band 8 mm wide; the console's USB pair hand-routed on
  F.Cu over In1 (U5's channels in the pair's order), EN's capacitor at
  the module's pin; reliefs on both pads of C2, C10, R3, C11-C14; notes
  corrected, the outputs sheet on A2.
- The PESD2CAN kept and documented (no stocked CAN TVS stays off at
  29.4 V and clamps under +40 V).

Bay node:
- SW3 placed on its pegs (-0.55 mm, Shouhan's land pattern); 2.2k I2C
  pull-ups; POS_IN 470k; AUX_VREF 1k; 100k on SVC; U9's input on a +5V
  island with three vias, C20 at its pins; C12 relieved; the camera note
  and the catalog's MPN text corrected.

Both re-routed: ERC 0, DRC 0 (the known C8 silkscreen warning), parity
0; CPL audit against JLC's footprints: every part agrees but SW3's pads
(0.13 mm, on purpose).  Bring-up measurements in assembly.md, the
resolution in pcba-review.md.

Co-Authored-By: Claude Opus 5.5 <noreply@anthropic.com>
Connections:
- net USB_CONN_DN: now also U5.4 (I/O2); no longer U5.6 (I/O1)
- net USB_CONN_DP: now also U5.6 (I/O1); no longer U5.4 (I/O2)
- net USB_DN: now also U5.3 (I/O2); no longer U5.1 (I/O1)
- net USB_DP: now also U5.1 (I/O1); no longer U5.3 (I/O2)
Changed lines of the file:
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@@
 		)
 	)
-	(label "USB_DN"
+	(label "USB_DP"
 		(at 113.03 248.92 180)
 		(fields_autoplaced yes)
@@
 		)
 	)
-	(label "USB_DP"
+	(label "USB_DN"
 		(at 113.03 251.46 180)
 		(fields_autoplaced yes)
@@
 		)
 	)
-	(label "USB_CONN_DP"
+	(label "USB_CONN_DN"
 		(at 128.27 251.46 0)
 		(fields_autoplaced yes)
@@
 		)
 	)
-	(label "USB_CONN_DN"
+	(label "USB_CONN_DP"
 		(at 128.27 248.92 0)
 		(fields_autoplaced yes)
@@
 		)
 	)
-	(text_box "GPIO: IO1/2/4/5 IMON A–D, IO6 VBUS_SENSE (ADC1) · IO7/8/9 CAN TX/RX/STB · IO10–13 POS A–D ·\n  IO14–17 ROW_EN A–D · IO18/21/47/33 FLT A–D · IO39 PD_INT, IO40/41 PD_SCL/SDA, IO42 I2C_PU · IO35 CTL LED ·\n  IO19/20 USB.  Strapping IO3/45/46 unused.\nTermination: two split 2 × 56 Ω + 4.7 nF (56 Ω in all) at the star centre; nodes carry none.\n+5V: buck (5.24 V; ≈ 4.8 V in dropout on a 5 V contract) or USB VBUS through B5819W Schottkys;\n  AP2112K (250 mV dropout) keeps 3.3 V down to a 5 V contract.  The TJA1462AT wants 4.5–5.5 V: CAN runs once VRACK is up."
+	(text_box "GPIO: IO1/2/4/5 IMON A–D, IO6 VBUS_SENSE (ADC1) · IO7/8/9 CAN TX/RX/STB · IO10–13 POS A–D ·\n  IO14–17 ROW_EN A–D · IO18/21/47/33 FLT A–D · IO39 PD_INT, IO40/41 PD_SCL/SDA, IO42 I2C_PU · IO35 CTL LED ·\n  IO19/20 USB.  Strapping IO3/45/46 unused.\nTermination: two split 2 × 56 Ω + 22 nF (56 Ω in all) at the star centre; nodes carry none.\n+5V: buck (5.24 V; ≈ 4.8 V in dropout on a 5 V contract) or USB VBUS through B5819W Schottkys;\n  AP2112K (250 mV dropout) keeps 3.3 V down to a 5 V contract.  The TJA1462AT wants 4.5–5.5 V: CAN runs once VRACK is up."
 		(exclude_from_sim no)
 		(at 20.32 386.08 0)
