File: electronics/data-port-x4/port1.kicad_sch (KiCad schematic)
At the start: 16 parts, among them J101 PORT1, J102 AUX1, U101 TPS2553DBVR-1, U102 INA226AIDGSR, U103 USBLC6-2SC6

Commit message: DATA ×4: the lead's D+/D− follow J7, the upstream pair rerouted
The node's J7 now has D+ on pin 3 and D− on pin 4 (094341c); the lead
mirrors pins (n ↔ 9 − n), so J1 takes D− on pin 5 and D+ on pin 6, like
the single DATA port's J2.  The upstream pair is drawn again without a
crossover: two vias in front of J1 (D+ north of D−), B.Cu west, north
along x 87 (clear of In2's +3V3 edge), west and south into the hub's top
pins; every turn keeps D+ on the pair's right, west of D− at the hub.

The new route moved the router's vias, and two of them cut In2's +5V in
half under the hub's capacitors: the +3V3 tab there ends at y 21.6 and a
via-only keep-out (pcbgen keepouts "vias_only") keeps the 1.9 mm +5V neck
whole.  The 22 µF VBUS caps' LCSC/MPN fields now reach the schematic and
the PCB too.  Docs: the lead pinout row.

ERC 0, DRC 0 (unconnected 0, parity 0); Konnect: 0 errors, the same three
library-copy warnings, JLC DFM 0.

Co-Authored-By: Claude Opus 5.5 <noreply@anthropic.com>
Parts:
- C102: LCSC (none) -> C45783; MPN (none) -> CL21A226MAQNNNE; Manufacturer (none) -> Samsung Electro-Mechanics
Changed lines of the file:
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@@
+			)
+		)
+		(property "LCSC" "C45783"
+			(at 139.7 90.17 0)
+			(effects
+				(font
+					(size 1.27 1.27)
+				)
+				(hide yes)
+			)
+		)
+		(property "MPN" "CL21A226MAQNNNE"
+			(at 139.7 90.17 0)
+			(effects
+				(font
+					(size 1.27 1.27)
+				)
+				(hide yes)
+			)
+		)
+		(property "Manufacturer" "Samsung Electro-Mechanics"
+			(at 139.7 90.17 0)
+			(effects
+				(font
+					(size 1.27 1.27)
+				)
+				(hide yes)
 			)
 		)

Commit message: DATA ×4: the PCBA review's fixes
X2: the lead's SDA, SCL and INT go through three 2N7002 (gate on this
board's +3V3, NXP AN10441) with 4.7k / 4.7k / 10k pull-ups on this side,
and the lead USBLC6s' VBUS pins are open: with DUT_5V off the node's
pull-ups no longer feed the dead board through the INA226 and TCA6408A
clamps.  X3: EN pulled down, every port off until the firmware enables
it.  X4: the Port netclass patterns get their leading *, VBUS and CC are
drawn at each receptacle (0.4 mm, no via on the CC lines), the INA226
reads Vbus on the shunt's sense pad, and R_ILIM sits beside its pin.  X5:
a shallow +3V3 tab and no via in the 2.5 mm +5V neck under the hub; the
bottom row's GND pads go on a bus to a via at each end.  X6: 100k
pull-ups on RESET and BOOT.  X7: TI's 1.45 mm exposed pad for the
TCA6408A.  X8: NON_REM0/1 pulled down.  X9: In2 notches keep the
upstream and PORT1 pairs over +5V all along; 100 nF at each port
USBLC6's VBUS.  X10: the crystal, PLLFILT and RBIAS drawn, no via.  X11
starts a bring-up measurement list in electronics.md.

The CPL audit agrees on all 106 parts (U3 and the new VQFN included).
Freerouting's few-µm dots on pads are dropped at import.  ERC 0, DRC 0,
parity 0, 0 unconnected; the BOM follows (about $104 for 5 with 2
assembled).

Co-Authored-By: Claude Opus 5.5 <noreply@anthropic.com>
Parts:
- added C104: 100n, Capacitor_SMD:C_0603_1608Metric, symbol Device:C
- added R109, R110: 100k, Resistor_SMD:R_0402_1005Metric, symbol Device:R
- R101: footprint Resistor_SMD:R_0603_1608Metric -> Resistor_SMD:R_0402_1005Metric; LCSC C25819 -> C25792; MPN 0603WAF4702T5E -> 0402WGF4702TCE
Connections:
- net +3V3: now also R109.1, R110.1; no longer R102.1
- net +5V: now also C104.1
- net GND: now also R102.2, C104.2
- net PORT1_BOOT_N: now also R110.2
- net PORT1_EN: now also R102.1; no longer R102.2
- net PORT1_RST_IO: now also R109.2
- net PORT1_SNS_N: now also U102.8 (Vbus)
- net PORT1_VBUS: no longer U102.8 (Vbus)
