File: electronics/data-port-x4/hub.kicad_sch (KiCad schematic)
At the start: 31 parts, among them J1 LEAD, U1 USB2514B-AEZC-TR, U2 TCA6408ARGTR, U3 AP2112K-3.3TRG1, U4 USBLC6-2SC6, U5 USBLC6-2SC6, U6 TCA6408ARGTR, Y1 X322524MSB4SI

Commit message: DATA ×4: the lead's D+/D− follow J7, the upstream pair rerouted
The node's J7 now has D+ on pin 3 and D− on pin 4 (094341c); the lead
mirrors pins (n ↔ 9 − n), so J1 takes D− on pin 5 and D+ on pin 6, like
the single DATA port's J2.  The upstream pair is drawn again without a
crossover: two vias in front of J1 (D+ north of D−), B.Cu west, north
along x 87 (clear of In2's +3V3 edge), west and south into the hub's top
pins; every turn keeps D+ on the pair's right, west of D− at the hub.

The new route moved the router's vias, and two of them cut In2's +5V in
half under the hub's capacitors: the +3V3 tab there ends at y 21.6 and a
via-only keep-out (pcbgen keepouts "vias_only") keeps the 1.9 mm +5V neck
whole.  The 22 µF VBUS caps' LCSC/MPN fields now reach the schematic and
the PCB too.  Docs: the lead pinout row.

ERC 0, DRC 0 (unconnected 0, parity 0); Konnect: 0 errors, the same three
library-copy warnings, JLC DFM 0.

Co-Authored-By: Claude Opus 5.5 <noreply@anthropic.com>
Connections:
- net UP_DN: now also J1.5 (Pin_5); no longer J1.6 (Pin_6)
- net UP_DP: now also J1.6 (Pin_6); no longer J1.5 (Pin_5)
Changed lines of the file:
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@@
 		)
 	)
-	(label "UP_DP"
+	(label "UP_DN"
 		(at 43.18 78.74 0)
 		(fields_autoplaced yes)
@@
 		)
 	)
-	(label "UP_DN"
+	(label "UP_DP"
 		(at 43.18 81.28 0)
 		(fields_autoplaced yes)

Commit message: DATA ×4: the PCBA review's fixes
X2: the lead's SDA, SCL and INT go through three 2N7002 (gate on this
board's +3V3, NXP AN10441) with 4.7k / 4.7k / 10k pull-ups on this side,
and the lead USBLC6s' VBUS pins are open: with DUT_5V off the node's
pull-ups no longer feed the dead board through the INA226 and TCA6408A
clamps.  X3: EN pulled down, every port off until the firmware enables
it.  X4: the Port netclass patterns get their leading *, VBUS and CC are
drawn at each receptacle (0.4 mm, no via on the CC lines), the INA226
reads Vbus on the shunt's sense pad, and R_ILIM sits beside its pin.  X5:
a shallow +3V3 tab and no via in the 2.5 mm +5V neck under the hub; the
bottom row's GND pads go on a bus to a via at each end.  X6: 100k
pull-ups on RESET and BOOT.  X7: TI's 1.45 mm exposed pad for the
TCA6408A.  X8: NON_REM0/1 pulled down.  X9: In2 notches keep the
upstream and PORT1 pairs over +5V all along; 100 nF at each port
USBLC6's VBUS.  X10: the crystal, PLLFILT and RBIAS drawn, no via.  X11
starts a bring-up measurement list in electronics.md.

The CPL audit agrees on all 106 parts (U3 and the new VQFN included).
Freerouting's few-µm dots on pads are dropped at import.  ERC 0, DRC 0,
parity 0, 0 unconnected; the BOM follows (about $104 for 5 with 2
assembled).

Co-Authored-By: Claude Opus 5.5 <noreply@anthropic.com>
Parts:
- added Q1, Q2, Q3: 2N7002, Package_TO_SOT_SMD:SOT-23, symbol Transistor_FET:2N7002
- added R5: 100k, Resistor_SMD:R_0603_1608Metric, symbol Device:R
- added R6, R7: 4.7k, Resistor_SMD:R_0402_1005Metric, symbol Device:R
- added R8: 10k, Resistor_SMD:R_0402_1005Metric, symbol Device:R
- U2, U6: footprint Package_DFN_QFN:QFN-16-1EP_3x3mm_P0.5mm_EP1.675x1.675mm -> Package_DFN_QFN:VQFN-16-1EP_3x3mm_P0.5mm_EP1.45x1.45mm
Connections:
- net +3V3: now also Q1.1 (G), Q2.1 (G), Q3.1 (G), R6.1, R7.1, R8.1; no longer U4.5 (VBUS), U5.5 (VBUS)
- net CFG_SEL0: now also U1.22 (SDA/SMBDATA/NON_REM1)
- net GND: now also R5.2
- net INT: now also Q3.2 (S), R8.2; no longer U5.1 (I/O1)
- net SCL: now also Q2.2 (S), R7.2; no longer U4.3 (I/O2)
- net SDA: now also Q1.2 (S), R6.2; no longer U4.1 (I/O1)
- net NON_REM0: now reaches U1.28 (SUSP_IND/LOCAL_PWR/NON_REM0)
- net NON_REM0: now also R5.1
- new net BUS_INT: Q3.3 (D), U5.1 (I/O1)
- new net BUS_SCL: Q2.3 (D), U4.3 (I/O2)
- new net BUS_SDA: Q1.3 (D), U4.1 (I/O1)
Other:
- note added: "I²C isolation: open with DUT_5V off, so the node's pull-ups cannot feed this board"

Commit message: DATA ×4: 100 × 37 mm, J1 at the rear end of the right edge, no fourth hole
On top of 1c0dfbd (100 × 28, J1 centred on the right edge):
- 100 × 37 mm, as deep as the v2: 13 mm deeper than the layout's 24 mm frame, still under JLC's 100 mm
  4-layer offer.
- J1 at the rear end of the right edge: mouth at drawer x 115, pins at drawer y 176–190, the plug
  (y ≈ 174–192) over the drawer's side window and clear of the v2's front-right boss. The LDO block
  and its islands sit in the corner behind it, unchanged.
- No fourth hole: v1 sits on H1–H3, unchanged in drawer coordinates, and on the front ledges. The
  plug forces stay in the board's plane. The drawer (2a3309b) already has no boss there.
- The upstream pair runs 45° from J1's vias into the hub's notch, and In2's +3V3 edge follows the
  diagonal: 16.7 / 17.2 mm pad to pin, 2 vias (1c0dfbd: 14.7 / 14.5). The lead's ESDs line up with
  J1's pins (flow-through). C13 and R2 move north of R5.

Against 1c0dfbd, unchanged or better:
- port pairs, their ESDs and the B.Cu lanes unchanged;
- every pair on one reference plane end to end (+5V on In2);
- +5V neck 2.45 mm (2.34);
- LDO islands unchanged (1.31 / 1.31 / 4.72 mm²);
- router copper 1580 mm (1612), signal vias 76 (79): the best of seven Freerouting variants. The 59
  extra GND vias are the larger pours' stitching.
- ERC 0, DRC 0, parity 0, 0 unconnected.
- CPL audit: 99 parts pass. The flags are the same 7 as 1c0dfbd's, positions agree: the USB4105s'
  symmetric pin 1, and the C1 / J1 / U3 land residuals against EasyEDA.

Worse:
- the upstream pair is 2.0 / 2.7 mm longer. J1's pins moved 6.4 mm to the rear, and a 45° route
  cannot do better (≈ 15 ps at 480 Mb/s, beside a 45 cm lead).
- its D+/D− mismatch is 0.53 mm (0.23). That is under the 1.27 mm usual for USB 2.0, and the
  downstream pairs already differ by 2.2 mm.

JLC's bare PCB at 100 × 37 (calculator, 2026-10-20): $13.10 for 5 ($8.00 offer + lead-free HASL
$5.10, no deburring line), $19.20 / $53.80 / $73.40 f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
Parts:
- removed H4: PT2.6, MountingHole:MountingHole_2.7mm_M2.5, symbol Mechanical:MountingHole
Changed lines of the file:
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@@
-	)
-	(symbol
-		(lib_id "Mechanical:MountingHole")
-		(at 548.64 215.9 0)
-		(unit 1)
-		(exclude_from_sim no)
-		(in_bom no)
-		(on_board yes)
-		(dnp no)
-		(fields_autoplaced yes)
-		(property "Reference" "H4"
-			(at 551.96 214.63 0)
-			(effects
-				(font
-					(size 1.27 1.27)
-				)
-			)
-		)
-		(property "Value" "PT2.6"
-			(at 553.535 217.17 0)
-			(effects
-				(font
-					(size 1.27 1.27)
-				)
-			)
-		)
-		(property "Footprint" "MountingHole:MountingHole_2.7mm_M2.5"
-			(at 548.64 215.9 0)
-			(effects
-				(font
-					(size 1.27 1.27)
-				)
-				(hide yes)
-			)
-		)
-		(property "Datasheet" ""
-			(at 548.64 215.9 0)
-			(effects
-				(font
-					(size 1.27 1.27)
-				)
-				(hide yes)
-			)
-		)
-		(property "Description" ""
-			(at 548.64 215.9 0)
-			(effects
-				(font
-					(size 1.27 1.27)
-				)
-				(hide yes)
-			)
-		)
-		(property "MPN" "M2.5 / PT 2.6 mounting hole"
-			(at 548.64 215.9 0)
-			(effects
-				(font
-					(size 1.27 1.27)
-				)
-				(hide yes)
-			)
-		)
-		(property "Manufacturer" "-"
-			(at 548.64 215.9 0)
-			(effects
-				(font
-					(size 1.27 1.27)
-				)
-				(hide yes)
-			)
-		)
-		(instances
-			(project "data-port-x4"
-				(path "/528ef17d-c8dc-5c1a-833a-a87b511a511e/5317ddbc-6eaf-528d-8064-6ad358d0599a"
-					(reference "H4")
-					(unit 1)
-				)
-			)
-		)
 	)
 	(symbol
