File: electronics/data-port-x4-v2/port4.kicad_sch (KiCad schematic)
At the start: 28 parts, among them J401 PORT4, J402 PINS4, U401 TPS2553DBVR-1, U402 INA226AIDGSR, U403 USBLC6-2SC6, U405 TPD4E05U06DQAR, U406 TPD4E05U06DQAR, U407 LSF0108RKSR

Commit message: DATA x4 v2: the H5VU25UC ESD and 22 ohm USB resistors, two extended types fewer, re-routed
The user's "essaie les 3 premiers ?", via the orchestrator: two part
swaps, each an extended part type less in the panel order.

- R23/R24, the RP2354B's USB series resistors: 27 ohm (C25100,
  extended) -> 22 ohm 0402 (C25092, basic).  The RP2350's USB is Full
  Speed only: its driver's own impedance plus 22 ohm stays inside USB's
  28-44 ohm driver window, nearer its middle than 33 ohm.  Said in
  design.py.
- U4, U105...U406, the nine 4-line ESD arrays: TI TPD4E05U06DQAR
  (C138714) -> hongjiacheng H5VU25UC (C20615800, JLC "preferred
  extended": no Economic fee; $0.03 against $0.08).
  - On its own DFN2510-10L land (the tools commit before this).
  - The same pins; its 6/7/9/10 are tied inside to 5/4/2/1, so the
    flow-through lines keep one signal.
  - Its stand-off is 5 V (TI's 5.5 V).  Every line it guards stays at
    5 V or less: a DUT's pins at its VREF (<= 5 V), the lead's I2C and
    INT at 3.3 V.
- The land changed (rows 0.875 mm apart, longer pads, a GND bar), so
  the board is re-routed: Freerouting at 4 layers, no neckdown, with one
  hand-drawn via under the RP2354B's exposed pad (that run left the pad
  unfanned).  Of the variants tried in parallel, the one with a single
  pad via closed every link; with four, its buses can't pass under the
  pad.  ERC 0, DRC 0 (4 silk warnings), 0 unconnected, parity 0.
- CPL: all nine H5VU25UC land pin by pin within 0.005 mm, pin 1 on
  pin 1 (JLC_CPL_FIX 270 degrees).  3D: 209 bodies resolve.
- Regenerated:
  - both variants' BOM/CPL;
  - the order panel (DRC 0; each half matches its variant; mouse
    bites unchanged);
  - the viewer's GLBs (gltfpack);
  - jlc_parts.json (C20615800 and C25092 added, nothing refreshed);
  - the BOM outputs.
- tools/bom.py, recomputed by the cost session's own method (components
  at the snapshot's breaks x 1.12, which reproduces the old figures
  exactly; JLC's library tier, so the H5VU2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
Parts:
- U405, U406: value TPD4E05U06DQAR -> H5VU25UC; footprint Package_SON:USON-10_2.5x1.0mm_P0.5mm -> bench:DFN2510-10L_2.5x1.0mm_P0.5mm; LCSC C138714 -> C20615800; MPN TPD4E05U06DQAR -> H5VU25UC; Manufacturer Texas Instruments -> hongjiacheng
Changed lines of the file:
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@@
 			)
 		)
-		(property "Value" "TPD4E05U06DQAR"
-			(at 70.85 309.88 0)
-			(effects
-				(font
-					(size 1.27 1.27)
-				)
-			)
-		)
-		(property "Footprint" "Package_SON:USON-10_2.5x1.0mm_P0.5mm"
+		(property "Value" "H5VU25UC"
+			(at 67.7 309.88 0)
+			(effects
+				(font
+					(size 1.27 1.27)
+				)
+			)
+		)
+		(property "Footprint" "bench:DFN2510-10L_2.5x1.0mm_P0.5mm"
 			(at 71.12 325.12 0)
 			(effects
@@
 			)
 		)
-		(property "Datasheet" "https://www.ti.com/lit/ds/symlink/tpd4e05u06.pdf"
+		(property "Datasheet" "https://wmsc.lcsc.com/wmsc/upload/file/pdf/v2/lcsc/2401261524_hongjiacheng-H5VU25UC_C20615800.pdf"
 			(at 71.12 325.12 0)
 			(effects
@@
 			)
 		)
-		(property "Description" "4-channel ESD, 0.5 pF, 5.5 V stand-off, flow-through (pins 6, 7, 9, 10 route through)"
+		(property "Description" "4-line ESD, 0.8 pF, 5 V stand-off, DFN2510-10L, flow-through (6, 7, 9, 10 tied to 5, 4, 2, 1)"
 			(at 71.12 325.12 0)
 			(effects
@@
 			)
 		)
-		(property "MPN" "TPD4E05U06DQAR"
+		(property "MPN" "H5VU25UC"
 			(at 71.12 325.12 0)
 			(effects
@@
 			)
 		)
-		(property "Manufacturer" "Texas Instruments"
+		(property "Manufacturer" "hongjiacheng"
 			(at 71.12 325.12 0)
 			(effects
@@
 			)
 		)
-		(property "LCSC" "C138714"
+		(property "LCSC" "C20615800"
 			(at 71.12 325.12 0)
 			(effects
@@
 			)
 		)
-		(property "Value" "TPD4E05U06DQAR"
-			(at 162.29 309.88 0)
-			(effects
-				(font
-					(size 1.27 1.27)
-				)
-			)
-		)
-		(property "Footprint" "Package_SON:USON-10_2.5x1.0mm_P0.5mm"
+		(property "Value" "H5VU25UC"
+			(at 159.14 309.88 0)
+			(effects
+				(font
+					(size 1.27 1.27)
+				)
+			)
+		)
+		(property "Footprint" "bench:DFN2510-10L_2.5x1.0mm_P0.5mm"
 			(at 162.56 325.12 0)
 			(effects
@@
 			)
 		)
-		(property "Datasheet" "https://www.ti.com/lit/ds/symlink/tpd4e05u06.pdf"
+		(property "Datasheet" "https://wmsc.lcsc.com/wmsc/upload/file/pdf/v2/lcsc/2401261524_hongjiacheng-H5VU25UC_C20615800.pdf"
 			(at 162.56 325.12 0)
 			(effects
@@
 			)
 		)
-		(property "Description" "4-channel ESD, 0.5 pF, 5.5 V stand-off, flow-through (pins 6, 7, 9, 10 route through)"
+		(property "Description" "4-line ESD, 0.8 pF, 5 V stand-off, DFN2510-10L, flow-through (6, 7, 9, 10 tied to 5, 4, 2, 1)"
 			(at 162.56 325.12 0)
 			(effects
@@
 			)
 		)
-		(property "MPN" "TPD4E05U06DQAR"
+		(property "MPN" "H5VU25UC"
 			(at 162.56 325.12 0)
 			(effects
@@
 			)
 		)
-		(property "Manufacturer" "Texas Instruments"
+		(property "Manufacturer" "hongjiacheng"
 			(at 162.56 325.12 0)
 			(effects
@@
 			)
 		)
-		(property "LCSC" "C138714"
+		(property "LCSC" "C20615800"
 			(at 162.56 325.12 0)
 			(effects

Commit message: DATA x4 v2: the usability review pass, layout B and a VBUS LED per port
One pass and one re-route for the usability review (docs/data-x4-logic-usability-review.md),
the user's go on layout B (2026-10-21):

- Layout B: one 2 × 6 per port, its pin names in two lines over it, the port number and the
  VBUS LED by its west end.  The headers sit 2 mm lower, at drawer z 28.5
  (rack.yaml › pcb.data_port_x4_v2.header), so the viewer's jumpers follow.
- A green VBUS LED per port (KT-0805G C2297 through 1k) on PORTn_5V_SW, before the shunt, so the
  INA226 doesn't count it.
- The LSF0108s' Vref_B/EN come from +5V_MX through 200k, not the port's VBUS, so each group is a
  voltage domain of its own.  The VREF dividers to the co-processor are 10k / 10k (were
  100k / 100k).  The bias current leaves by Vref_A: through 100k it would float an unwired VREF
  to about 2.1 V and the group would pass.  Through 10k it stays near 0.4 V, under the 0.65 V the
  LSF needs.  A board that is off isolates.
- The co-processor's AP2112K (U12) is out.  +3V3_CP comes from +3V3 through a 600 Ω ferrite
  (FB2, C1017).  U3 (AP2114H) then carries about 0.39 A, 0.66–0.75 W.
- Docs: the base solders two 2 × 1 pieces per port (GND/VREF, RESET/BOOT).

Re-routed with Freerouting (4 layers):
- ERC 0, copper DRC 0, 0 unconnected, parity 0.  The 4 silk-over-pad warnings are unchanged
  (U107–U407's marker on C105–C405).
- 216 3D models resolve.
- CPL: the new parts land within 0.1 mm rms, the LEDs placed by function.
- The cradle keep-outs clear by at least 0.67 mm: slots and latch, T-heads, rear band, boss.
  Checked in SolidCraft against the new STEP.

Regenerated:
- Both variants' BOM and CPL (base: 91 DNP).
- The order panel; its halves match their variants.
- The viewer GLBs and rack.json.

Cost, by the cost session's method in bom.py:
- The logic has 40 part types, 17 extended (was 41 and 18).
- The panel order of 2: $229.91 → $226.88 (−$3.03).
- Logic alone: $168.53 → $165.27.  Base alone: $84.50 → $8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
Parts:
- added D401: KT-0805G, LED_SMD:LED_0805_2012Metric, symbol Device:LED
- added R414: 1k, Resistor_SMD:R_0402_1005Metric, symbol Device:R
- R412, R413: value 100k -> 10k; LCSC C25741 -> C25744; MPN 0402WGF1003TCE -> 0402WGF1002TCE
Connections:
- net GND: now also D401.1 (K)
- net PORT4_5V_SW: now also R414.1
- net PORT4_VBUS: no longer R411.1
- new net +5V_MX: R411.1
- new net PORT4_LED_A: D401.2 (A), R414.2
Other:
- note added: "Header 4 (2 × 6 through-hole): GND, VREF, P1–P8, RESET_N, BOOT_N; RESET/BOOT through 1k, their expander lines pulled up"
- note removed: "Header 4 (2 × 6 SMD): GND, VREF, P1–P8, RESET_N, BOOT_N; RESET/BOOT through 1k, their expander lines pulled up"
