File: electronics/data-port-x4-v2/data-port-x4-v2.kicad_sch (KiCad schematic)
At the start: 0 parts

Commit message: DATA x4 v2: the base DATA-4x as an assembly variant, a 1 A 3.3 V LDO, re-routed
The user's call: v1 is not ordered for the proto ("pour la data 4x on
attend la version verticale"); the base DATA-4x is this board with the
logic left off.  One PCB, two assemblies:
- DATA-4x-logic, as drawn: fab/data-port-x4-v2-bom-jlcpcb.csv, -cpl-...
- DATA-4x, the base (b.pcb["variants"]["base"]): fab/data-port-x4-v2-base-
  bom-jlcpcb.csv, -base-cpl-jlcpcb.csv, data-port-x4-v2-base-bom.csv.
  92 parts off: the matrix and co-processor sheets whole, and each port's
  pin chain (TPD4E05U06 x2, the 100 ohm arrays, the LSF0108, its Vref_B
  and VREF parts).  24 part types (10 extended), 112 parts, 511 joints.

The base checked against v1's functions and review fixes (the DATA x4
session's list): the hub; the four ports with switch, R_ILIM, INA226,
USBLC6, CC and bulk; the expanders with RESET/BOOT; the lead's ESD and
I2C isolation; the 3.3 V.  No base signal passes through a logic part,
so no 0 ohm or solder jumper: the headers' GND/RESET/BOOT stay live,
hub port 5 ends on R23/R24's empty pads (ports 5-7 left enabled, as the
logic board's 6-7).

The review's other points:
- U3: the USB2517I draws 330 mA with four High-Speed ports (datasheet,
  typical), 0.6-0.7 W from 5.0-5.24 V: too much for v1's AP2112K in
  SOT-23-5.  Now an AP2114H-3.3 (SOT-223, 1 A, 0.16 V dropout at 0.35 A,
  as v1 wants the hub to outlive a sagging +5V), its tab on a top-side
  +3V3 island with six vias into the plane, VIN on a +5V island with two;
  22 uF 0805 in and out.  The AMS1117 would save $3.07 but drops 1.1 V.
- C1 (J1's bulk) 22 uF in 1206, as v1.
- The routed +5V at 0.6 mm (Power), as v1.  The ports' 5V_SW and VBUS
  stay at 0.3 mm: the vertical USB-C's VBUS pads are 0.3 mm wide at a
  0.5 mm pitch; 15 mm of it drops ~15 mV at the 0.62 A limit.
- HASL for the base ordered alone: a pricing note ($12 less).

Re-routed by Freerouting at 4 layers, no neckdown; CP_RUN (the matrix
expander to the co-processo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
Changed lines of the file:
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@@
 		)
 	)
-	(text_box "DATA ×4 v2.0 — USB2517I hub (7 ports), four USB-C (sub-slots A1.1–A1.4) each with a TPS2553-1, an INA226\n  and ESD, two TCA6408A for EN/FAULT/RESET/BOOT, an AP2112K 3.3 V; the PH 8 lead from the node's J7.\nPins: 32 on two CH446Q (±5 V), LSF0108 per port, an RP2354B analyzer on hub port 5, a TCA9534A for\n  the matrix and the co-processor's RUN/BOOTSEL.  Standing behind the port wall, one face assembled;\n  v1 stays the other bays' board.\nLead pinout here: 1 INT · 2 SCL · 3 SDA · 4 GND · 5 D− · 6 D+ · 7 GND · 8 +5V (the node's J7 mirrored).\nI²C: TCA6408A 0x20 / 0x21, INA226 0x41 / 0x43 / 0x44 / 0x45, TCA9534A 0x38; the node's INA226 0x40."
+	(text_box "DATA ×4 v2.0 — USB2517I hub (7 ports), four USB-C (sub-slots A1.1–A1.4) each with a TPS2553-1, an INA226\n  and ESD, two TCA6408A for EN/FAULT/RESET/BOOT, an AP2114H 3.3 V; the PH 8 lead from the node's J7.\nPins: 32 on two CH446Q (±5 V), LSF0108 per port, an RP2354B analyzer on hub port 5, a TCA9534A for\n  the matrix and the co-processor's RUN/BOOTSEL.  Standing behind the port wall, one face assembled;\n  v1 stays the other bays' board.\nLead pinout here: 1 INT · 2 SCL · 3 SDA · 4 GND · 5 D− · 6 D+ · 7 GND · 8 +5V (the node's J7 mirrored).\nI²C: TCA6408A 0x20 / 0x21, INA226 0x41 / 0x43 / 0x44 / 0x45, TCA9534A 0x38; the node's INA226 0x40.\nAssembled as DATA-4x-logic (as drawn) or DATA-4x (BOM/CPL '-base': the matrix, the co-processor and the\n  ports' pin chains not fitted)."
 		(exclude_from_sim no)
 		(at 30 267.97 0)
-		(size 534 21.59)
+		(size 534 25.4)
 		(margins 2 2 2 2)
 		(stroke

Commit message: DATA x4 v2: the usability review pass, layout B and a VBUS LED per port
One pass and one re-route for the usability review (docs/data-x4-logic-usability-review.md),
the user's go on layout B (2026-10-21):

- Layout B: one 2 × 6 per port, its pin names in two lines over it, the port number and the
  VBUS LED by its west end.  The headers sit 2 mm lower, at drawer z 28.5
  (rack.yaml › pcb.data_port_x4_v2.header), so the viewer's jumpers follow.
- A green VBUS LED per port (KT-0805G C2297 through 1k) on PORTn_5V_SW, before the shunt, so the
  INA226 doesn't count it.
- The LSF0108s' Vref_B/EN come from +5V_MX through 200k, not the port's VBUS, so each group is a
  voltage domain of its own.  The VREF dividers to the co-processor are 10k / 10k (were
  100k / 100k).  The bias current leaves by Vref_A: through 100k it would float an unwired VREF
  to about 2.1 V and the group would pass.  Through 10k it stays near 0.4 V, under the 0.65 V the
  LSF needs.  A board that is off isolates.
- The co-processor's AP2112K (U12) is out.  +3V3_CP comes from +3V3 through a 600 Ω ferrite
  (FB2, C1017).  U3 (AP2114H) then carries about 0.39 A, 0.66–0.75 W.
- Docs: the base solders two 2 × 1 pieces per port (GND/VREF, RESET/BOOT).

Re-routed with Freerouting (4 layers):
- ERC 0, copper DRC 0, 0 unconnected, parity 0.  The 4 silk-over-pad warnings are unchanged
  (U107–U407's marker on C105–C405).
- 216 3D models resolve.
- CPL: the new parts land within 0.1 mm rms, the LEDs placed by function.
- The cradle keep-outs clear by at least 0.67 mm: slots and latch, T-heads, rear band, boss.
  Checked in SolidCraft against the new STEP.

Regenerated:
- Both variants' BOM and CPL (base: 91 DNP).
- The order panel; its halves match their variants.
- The viewer GLBs and rack.json.

Cost, by the cost session's method in bom.py:
- The logic has 40 part types, 17 extended (was 41 and 18).
- The panel order of 2: $229.91 → $226.88 (−$3.03).
- Logic alone: $168.53 → $165.27.  Base alone: $84.50 → $8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
Other:
- note added: "+5V_MX"
- note added: "-5V, BUS_A/B/C/D/E/F/G/H,"
- note added: "CP_BOOT_N, CP_RUN, MARK"
- note removed: "+5V_MX, -5V,"
- note removed: "BUS_A/B/C/D/E/F/G/H, CP_BOOT_N,"
- note removed: "CP_RUN, MARK"

Commit message: DATA x4 v2: D2 holds the co-processor in reset with the hub (schematic review S2)
With CFG_SEL 000 the USB2517 samples each downstream D+ / D- as a
port-disable strap when RESET_N rises, and one high line disables the
port (DS00001598C Table 5-1 p.10, checked by the user): the RP2354B's
D+ pull-up on port 5 must not be up by then.

- D2, one Schottky of a BAT54S (C7420333, preferred, no fee; VF <= 240 mV
  at 0.1 mA, <= 320 mV at 1 mA) from CP_RUN to HUB_RST_N, on both
  variants (its second diode open).  RUN sits at ~0.3 V while RESET_N is
  low (R25's ~0.33 mA), under the RP2350's VIL 0.8 V.
- R25 now also charges C6: the hub's reset to VIH 2.0 V goes from ~9.3 to
  ~4.6-5 ms, >> the 1 us minimum; RESET_N stays under VIL through a 3.3 V
  rise of up to ~1.3 ms (DS Note 8-1).
- electronics.md: a self-powered DUT attached during the hub's reset
  loses its port until the next hub reset; CFG_SEL 110 (internal
  defaults, straps off) studied as a way out, not applied, pending the
  user's reading (datasheet audit U11, U12).
- Placed and routed from the vetted routing as a seed, tidy pass, DRC and
  ERC clean; schematics, BOMs, CPL, Gerbers, panel, renders, GLBs.
- bom.py: the BAT54S as added since the panel's quote ($207.89 for 2).

Co-Authored-By: Claude Opus 5.5 <noreply@anthropic.com>
Other:
- note added: "CP_BOOT_N, MARK"
- note added: "CP_RUN"
- note removed: "CP_BOOT_N, CP_RUN, MARK"

Commit message: DATA x4 v2: datasheet audit fixes 1-9, conservative options, CFG_SEL 110
The DATA x4 v2 datasheet audit's fixes, approved by the user, plus the
conservative options that close U2, U8, U9 and U10:

- Core regulator (fixes 1-3).
  - L1 on a polarity-marked land: bench:L_Abracon_AOTA-B201610, RP's
    0.7 x 1.7 mm pads, the dot on pad 1 = +1V1 (U1's answer).
  - The block is Raspberry Pi's RP2350B Minimal R4-S1 one, turned 180
    degrees with U11, at their coordinates.  CIN and COUT sit on RP's
    0402 land (bench:C_0402_1005Metric_RP), so LX runs 0.3 mm between
    them.
  - Copper: their F.Cu areas (LX, +1V1 with the two V_OUT vias, PGND
    with its two vias, VIN) and their settings; VREG_FB taken at the
    V_OUT vias; CFILT on its own via.
  - The F.Cu GND pour leaves a hole round the block, so PGND meets the
    main GND only through its two vias.  No copper under LX and L1 on
    In1, In2 and B.Cu.
- Fix 4: C47 (DVDD pin 32) 100 nF -> 4.7 uF.
- Fix 5: R40 47k -> 10k, so GPIO45 stays >= -0.48 V; formula updated.
- Fix 6: UMW MAX809S (U5, C347371) drives the hub's RESET_N in place of
  R2/C6; C6 is its 100 nF.
- Fix 7: two H5VU25UC per port in flow-through.  VREF and RESET/BOOT
  sit at the header's two ends, so one part per end:
  - U108-U408 take VREF (logic only);
  - U109-U409 take RESET_N/BOOT_N with the 1k right behind them, fitted
    on the base too (schematic review N4).
  VREF and ports 1-3's RESET_N are drawn into their ESD pins; all 12
  lines checked in flow-through.
- Fixes 8, 9: the VREF isolation wording and the firmware rule (switches
  open below 0.65 V, in multi-dut-node.md); +5V_MX ~1-4 mA, FB1 and U3
  stale lines gone.
- Conservative options:
  - U2: R10 1M across XI-XO (C26083);
  - U8: R115-R415 100k in series with GPIO40-43;
  - U9: R11, R12 10k on the TCA6408A RESETs;
  - U10: C7, C8 4.7 uF.
- Hub on CFG_SEL 110, internal defaults with straps disabled (U11, U12
  answered by the user).  CFG_SEL1 and CFG_SEL2 pull up through their
  RN2/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
Other:
- note added: "CP_ADC1"
- note added: "CP_ADC2"
- note added: "CP_ADC3"
- note added: "CP_ADC4"
- note added: "CP_BOOT_N, CP_RUN, MARK"
- note removed: "CP_BOOT_N, MARK"
- note removed: "CP_RUN"
- note removed: "CP_VREF1"
- note removed: "CP_VREF2"
- note removed: "CP_VREF3"
- note removed: "CP_VREF4"
