File: electronics/data-port-x4-v2-6l/hub.kicad_sch (KiCad schematic)
At the start: 41 parts, among them J1 LEAD, Q1 2N7002, Q2 2N7002, Q3 2N7002, U1 USB2517I-JZX, U2 TCA6408ARGTR, U3 AP2114H-3.3TRG1, U4 H5VU25UC, U6 TCA6408ARGTR, Y1 X322524MSB4SI

Commit message: DATA x4 v2: the rack's board on 4 layers again, the 6-layer build kept
The user's choice, now that the routing portfolio and its fixes route it
clean: JLC04161H-7628 (F, GND, power, B), cheaper and faster than 6.

- config pcb.data_port_x4_v2.layers is 4.  electronics/data-port-x4-v2 is
  rebuilt on 4 layers and routed with run ripup30-order2's session: 750 vias,
  5194 mm, 1930 bends; 0 open, copper DRC 0, parity 0, ERC 0.  Its only vias
  in pads are the 8 in the QFNs' thermal pads, accepted unfilled.
- The order panel (a logic and a base, 100 x 142 mm) is regenerated from it:
  4 layers, ENIG, both halves matching their variants.
- The 6-layer board moves to electronics/data-port-x4-v2-6l, its routing
  unchanged, behind a design.py that builds the design with X4V2_LAYERS=6.
  The 4-layer folder it replaces (data-port-x4-v2-4l) is gone; the Hardware
  CI checks the -6l instead.
- Regenerated: Gerbers, renders, the panel's, the viewer's models of both
  variants; BOM, CPL and schematics are unchanged.
- Docs: the stackup is 4 layers again, with the why, the finish (ENIG for the
  panel and the logic, lead-free HASL for a base alone), the vias in pads and
  JLC's 4-layer prices; the benchmark's status.  tools/bom.py and bom/ are
  left to the pricing update.

Co-Authored-By: Claude Opus 5.5 <noreply@anthropic.com>
Other:
- title: DATA ×4 v2, 4 layers — Lead, hub, expanders, 3.3 V -> DATA ×4 v2 — Lead, hub, expanders, 3.3 V
