File: electronics/bay-node/bay-node.kicad_pcb (KiCad board)
At the start: 4 copper layers, 74 x 90 mm, 105 parts, among them J1 ROW IN, J2 ROW OUT, J3 PC, J5 AUX, J6 CAM, J7 DATA, Q1 SUD50P06-15(UMW), Q2 2N7002, Q3 2N7002, Q4 AO3400A, SW1 RESET, SW2 BOOT, SW3 SERVICE, U1 LMR51625YDDCR, U10 INA226AIDGSR, U11 TJA1462AT, U12 USBLC6-2SC6, U13 USBLC6-2SC6, U2 AP2114H-3.3TRG1, U3 ESP32-S3-WROOM-1-N8R8, U4 USBLC6-2SC6, U5 MUX_PC, U6 MUX_DUT, U7 SN74LVC1G32DBVR, U8 USBLC6-2SC6, U9 TPS2553DDBVR

Commit message: Datasheet audit F1-F6: the pod's AP2114H, STB 5.1k, PC_DET hysteresis, the camera ESD's 100 nF, the eFuse step
The user approved the audit's fixes for the node, the hub and the pod
("Go pour 1"); docs/datasheet-audit.md marks F1-F6 applied.

* F1, camera pod: U1 AMS1117-3.3 -> AP2114H-3.3TRG1 (C150716, catalog
  ldo_1a, the node's U2).
  - The AMS1117 is specified stable only with 22 uF tantalum; the
    AP2114H is stable with the ceramic C2.
  - Same SOT-223 pinout, copper (the +3V3 pour and island round the
    tab stay) and 180 deg CPL correction.
  - One more extended type on the pod's Economic order: +$3.09 and
    $0.05 of parts (JLC_SINCE_QUOTE).
* F2, power hub: R214 (TJA1462 STB pull-down) 10k -> 5.1k (C23186,
  already on the board). With IO9 floating, STB's internal pull-up
  (20 kOhm minimum) left it at up to 1.10 V, over VIL 0.99 V.
* F3, bay node: R42 150k from MUX_SEL back to PC_DET, beside U7 (C22807,
  on the board since S1).
  - The laptop's VBUS rises at ~50 us/V through R11/R12, where the
    LVC1G32 wants <= 10 ns/V and warns of oscillation.
  - This gives ~0.14 V of hysteresis.
* F4, bay node: C28 100 nF (C14663) on U12/U13's VBUS pins (+3V3), above
  U12 by its pin 5. Between the two ICs their courtyards leave no room.
* F5, node and hub: firmware.md's first-flash procedure gains the
  irreversible DIS_USB_OTG_DOWNLOAD_MODE eFuse step. In USB-OTG
  download boot the ROM drives IO40 high: the node's DUT_FLT_N, the
  hub's PD_SCL. Nothing is burnt.
* F6, notes, hub:
  - the IMON filter is 0.9 ms, not 47 us: the pin is a current source;
  - the buck stops at ~3.8 V (internal UVLO);
  - SHDN turns on at >= 1 V;
  - the soft start stays under the limit only typically;
  - the CH224A note follows CH224 V2.1: the source PDOs are listed for
    both parts and readable under 100 W, which is still to check with
    ours (review R3); single-byte transfers; no "same die".
* F6, notes, node: TPS2553D; the LDO's 1.94 V x 0.4 A ~ 0.8 W; L1's
  7.5 A guarante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
Parts:
- added C28: 100n, Capacitor_SMD:C_0603_1608Metric, F.Cu at (53.6, 13.2)
- added R42: 150k, Resistor_SMD:R_0603_1608Metric, F.Cu at (24.4, 42.0)
Routing:
- net POS_IN: track 75.2 -> 108.0 mm, vias 0 -> 2
- net CAM_CS: track 46.1 -> 71.9 mm, vias 3 -> 2
- net /USB/MUX_SEL: track 22.8 -> 34.0 mm
- net /Camera/CAM_SCK_C: track 15.9 -> 27.0 mm
- net POS_OUT: track 73.2 -> 82.9 mm, vias 2 -> 4
- net I2C_SCL: track 58.3 -> 49.0 mm, vias 7 -> 0
- net I2C_SDA: track 62.8 -> 53.9 mm, vias 2 -> 4
- net DUT_EN: track 49.2 -> 57.8 mm
- net SVC: track 98.0 -> 105.7 mm
- net AUX_TX: track 42.6 -> 35.5 mm, vias 4 -> 2
- net /MCU/LED_DIN: track 90.5 -> 97.6 mm, vias 4 -> 2
- net /Camera/CAM_MOSI_C: track 28.0 -> 34.9 mm, vias 3 -> 0
- net CAM_LED: track 51.3 -> 44.7 mm
- net /DUT power & AUX/SHUNT_P: track 24.8 -> 31.3 mm
- net CAN_H: track 76.7 -> 83.3 mm, vias 3 -> 4
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