File: electronics/bay-node/bus.kicad_sch (KiCad schematic)
At the start: 9 parts, among them U11 TCAN1462V

Commit message: CAN transceiver: the TJA1462AT on the hub and the node
The TCAN1462V (C7399456) had no LCSC stock on 2026-10-18 and 19, and
JLC's quote of the hub asked for another part.  The user chose NXP's
TJA1462AT/0Z (C3234095, 10 500 in stock) for both boards (hub U6, node
U11): the same SOIC-8 pinout (VIO on pin 5, STB on pin 8), signal
improvement kept, bus pins -36/+40 V instead of ±58 V.  The TCAN1462V
and the TCAN1044AV stay the alternates.

Both boards regenerated and the same Freerouting sessions re-imported
(tracks and vias unchanged): ERC 0, DRC 0 errors (the hub's known C8
silkscreen warning), 0 unconnected, parity 0, JLC READY.  The CPL keeps
its 270° correction (C3234095 was already in build_board.py).

Docs: can.md, electronics.md, firmware comments and pin tables,
bom/sourcing.md, which also notes that JLC unticks the USB4105 (hard to
process, $0.03 a piece): tick it again at every order.

Co-Authored-By: Claude Opus 5.5 <noreply@anthropic.com>
Parts:
- U11: value TCAN1462V -> TJA1462AT; Alternative LCSC stock was 0 on 2026-10-18. Same pinout: TCAN1044AVDRQ1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 -> Same pinout: TI TCAN1462VDRQ1 (C7399456, SIC, bus pins ±58 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; LCSC C7399456 -> C3234095; MPN TCAN1462VDRQ1 -> TJA1462AT/0Z; Manufacturer Texas Instruments -> NXP Semiconductors
Other:
- note added: "CAN: TJA1462AT on the row pair (J1.3/4 ↔ J2.4/3, Power sheet); stub ≤ 20 mm, no termination"
- note removed: "CAN: TCAN1462V on the row pair (J1.3/4 ↔ J2.4/3, Power sheet); stub ≤ 20 mm, no termination"
Changed lines of the file:
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@@
 			)
 		)
-		(property "Value" "TCAN1462V"
+		(property "Value" "TJA1462AT"
 			(at 86.005 34.29 0)
 			(effects
@@
 			)
 		)
-		(property "Datasheet" "https://www.ti.com/lit/ds/symlink/tcan1462-q1.pdf"
+		(property "Datasheet" "https://www.nxp.com/docs/en/data-sheet/TJA1462.pdf"
 			(at 91.44 45.72 0)
 			(effects
@@
 			)
 		)
-		(property "Description" "CAN FD SIC transceiver, VCC 5 V, VIO 1.7–5.5 V, bus pins ±58 V (MCP2562 pinout)"
+		(property "Description" "CAN FD SIC transceiver, VCC 5 V, VIO 2.95–5.5 V, bus pins −36/+40 V (MCP2562 pinout)"
 			(at 91.44 45.72 0)
 			(effects
@@
 			)
 		)
-		(property "MPN" "TCAN1462VDRQ1"
+		(property "MPN" "TJA1462AT/0Z"
 			(at 91.44 45.72 0)
 			(effects
@@
 			)
 		)
-		(property "Manufacturer" "Texas Instruments"
+		(property "Manufacturer" "NXP Semiconductors"
 			(at 91.44 45.72 0)
 			(effects
@@
 			)
 		)
-		(property "LCSC" "C7399456"
+		(property "LCSC" "C3234095"
 			(at 91.44 45.72 0)
 			(effects
@@
 			)
 		)
-		(property "Alternative" "LCSC stock was 0 on 2026-10-18.  Same pinout: TCAN1044AVDRQ1 (C3234993, no SIC, ±58 V) or NXP TJA1462AT/0Z (C3234095, SIC, VIO 2.95–5.5 V, bus pins −36/+40 V)"
+		(property "Alternative" "Same pinout: TI TCAN1462VDRQ1 (C7399456, SIC, bus pins ±58 V; LCSC stock 0 on 2026-10-18 and 19) or TCAN1044AVDRQ1 (C3234993, no SIC, ±58 V)"
 			(at 91.44 45.72 0)
 			(effects
@@
 		)
 	)
-	(text "CAN: TCAN1462V on the row pair (J1.3/4 ↔ J2.4/3, Power sheet); stub ≤ 20 mm, no termination"
+	(text "CAN: TJA1462AT on the row pair (J1.3/4 ↔ J2.4/3, Power sheet); stub ≤ 20 mm, no termination"
 		(exclude_from_sim no)
 		(at 16.51 17.78 0)
@@
 		)
 	)
-	(text_box "CAN (docs/can.md): one bus for the rack, a star from the hub; both terminations sit in the hub.\n  250 kbit/s (125 kbit/s fallback).  TCAN1462V (SIC): VCC 5 V, VIO 3.3 V, bus pins ±58 V, passive unpowered.\nPOS: active-high 3.3 V token.  From reset the node holds POS_OUT low; when POS_IN goes high and it has\n  no address yet, it answers with its MAC, takes (row, position) from the hub, then raises POS_OUT.\n  R29 keeps POS_IN low with no cable; the next node's 100k keeps POS_OUT low before firmware."
+	(text_box "CAN (docs/can.md): one bus for the rack, a star from the hub; both terminations sit in the hub.\n  250 kbit/s (125 kbit/s fallback).  TJA1462AT (SIC): VCC 5 V, VIO 3.3 V, bus pins −36/+40 V, passive unpowered.\nPOS: active-high 3.3 V token.  From reset the node holds POS_OUT low; when POS_IN goes high and it has\n  no address yet, it answers with its MAC, takes (row, position) from the hub, then raises POS_OUT.\n  R29 keeps POS_IN low with no cable; the next node's 100k keeps POS_OUT low before firmware."
 		(exclude_from_sim no)
 		(at 15.24 177.8 0)

Commit message: PCBA review: hub and node fixes before the order
On main's CH224A hub and the bay node v0.5.

Power hub:
- CPL: the side LEDs (C598310, C4555382) +0.825 mm, their polarity
  proven from JLC's own footprints (and C495809 at 270 deg in the table,
  for the IRF7842 the AP33772S hub had).
- Rows: SHDN pull-downs 10k, so rows stay off without firmware (100k
  gave 1 V at the pin's 10 uA); a B5819W at each row output for the
  cable's kick; the red FAULT LEDs fed from their ROW_EN, so a row that
  is simply off shows no fault.
- In2's VRACK band 8 mm wide; the console's USB pair hand-routed on
  F.Cu over In1 (U5's channels in the pair's order), EN's capacitor at
  the module's pin; reliefs on both pads of C2, C10, R3, C11-C14; notes
  corrected, the outputs sheet on A2.
- The PESD2CAN kept and documented (no stocked CAN TVS stays off at
  29.4 V and clamps under +40 V).

Bay node:
- SW3 placed on its pegs (-0.55 mm, Shouhan's land pattern); 2.2k I2C
  pull-ups; POS_IN 470k; AUX_VREF 1k; 100k on SVC; U9's input on a +5V
  island with three vias, C20 at its pins; C12 relieved; the camera note
  and the catalog's MPN text corrected.

Both re-routed: ERC 0, DRC 0 (the known C8 silkscreen warning), parity
0; CPL audit against JLC's footprints: every part agrees but SW3's pads
(0.13 mm, on purpose).  Bring-up measurements in assembly.md, the
resolution in pcba-review.md.

Co-Authored-By: Claude Opus 5.5 <noreply@anthropic.com>
Parts:
- R29: value 100k -> 470k; LCSC C25803 -> C23178; MPN 0603WAF1003T5E -> 0603WAF4703T5E
Changed lines of the file:
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@@
 			)
 		)
-		(property "Value" "100k"
+		(property "Value" "470k"
 			(at 93.016 114.3 0)
 			(effects
@@
 			)
 		)
-		(property "Description" "Resistor 100k 0603"
+		(property "Description" "Resistor 470k 0603"
 			(at 88.9 113.03 0)
 			(effects
@@
 			)
 		)
-		(property "LCSC" "C25803"
+		(property "LCSC" "C23178"
 			(at 88.9 113.03 0)
 			(effects
@@
 			)
 		)
-		(property "MPN" "0603WAF1003T5E"
+		(property "MPN" "0603WAF4703T5E"
 			(at 88.9 113.03 0)
 			(effects

Commit message: Bay node: AP2114H for the 3.3 V, camera ESD clamped to +3V3
The schematic counter-review's fixes, approved by the user.

- U2: AP2114H-3.3TRG1 (C150716, catalog ldo_1a) instead of the AMS1117-3.3.
  It is specified stable with ceramics (C11, C12); the AMS1117 guarantees it
  only with 22 uF tantalum.  Same SOT-223 "H" pinout (1 GND, 2 and tab VOUT,
  3 VIN), footprint and copper: only the part's properties change.
- U12, U13 (USBLC6 on the camera lead): pin 5 on +3V3 instead of CAM_5V.
  With CAM_5V off (the PTC tripped), the SPI lines would feed the pod through
  the upper diodes, and CAM_5V's clamp sits above the ESP32's 3.6 V.  A
  minimal patch of the routing, no re-route: the CAM_5V stub that only
  reached the two pins goes (10 segments); U12.5 gets a +3V3 feed to a via in
  In2's +3V3 area; U13.5, with no room for its own, joins U12.5 along the
  stub's old east path at 0.25 mm.  The straightening pass ran on +3V3 and
  CAM_5V.
- Stale notes: AUX_VREF goes through R23's 1k, not 33 ohms; the next node's
  pull-down is R29's 470k, not 100k.
- pcbgen.fanout_pads takes `only` (REF.PAD), to fan out a few pads of a
  routed board.

ERC 0, DRC 0, unconnected 0, parity 0, every 3D model found.  The renders,
Gerbers and viewer model are regenerated (the unchanged iso render kept).
The schematic, the BOM and the docs (the node table, the CPL fix table, the
bring-up check, PCBA review N9) follow.  The hub and bom/ are untouched.

Co-Authored-By: Claude Opus 5.5 <noreply@anthropic.com>
Changed lines of the file:
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@@
 		)
 	)
-	(text_box "CAN (docs/can.md): one bus for the rack, a star from the hub; both terminations sit in the hub.\n  250 kbit/s (125 kbit/s fallback).  TJA1462AT (SIC): VCC 5 V, VIO 3.3 V, bus pins −36/+40 V, passive unpowered.\nPOS: active-high 3.3 V token.  From reset the node holds POS_OUT low; when POS_IN goes high and it has\n  no address yet, it answers with its MAC, takes (row, position) from the hub, then raises POS_OUT.\n  R29 keeps POS_IN low with no cable; the next node's 100k keeps POS_OUT low before firmware."
+	(text_box "CAN (docs/can.md): one bus for the rack, a star from the hub; both terminations sit in the hub.\n  250 kbit/s (125 kbit/s fallback).  TJA1462AT (SIC): VCC 5 V, VIO 3.3 V, bus pins −36/+40 V, passive unpowered.\nPOS: active-high 3.3 V token.  From reset the node holds POS_OUT low; when POS_IN goes high and it has\n  no address yet, it answers with its MAC, takes (row, position) from the hub, then raises POS_OUT.\n  R29 keeps POS_IN low with no cable; the next node's 470k keeps POS_OUT low before firmware."
 		(exclude_from_sim no)
 		(at 15.24 177.8 0)

Commit message: Schematic review S1, S4, S6: POS_IN 150k, the hub's ON LEDs on 18k, the camera's 0.75 A PTC
The user approved them ("S1 oui / S6 oui / S4 oui").

* S1, bay node: R29 470k -> 150k (C22807, basic).
  - Before its firmware runs, the upstream POS output (a node's IO42, the
    hub's IO10-13) floats. The BAT54S's warm leakage (about 2-3 uA at
    65 C) could then lift POS_IN through 470k to VIL.
  - Driven high through R30 + R28, 150k still gives 2.87 V, above VIH.
  - The design.py notes and bay_node.dtsi follow.
* S4, power hub: R41-R44 (the ON LEDs on the row outputs) 10k -> 18k
  (C25810, already on the board): 1.4 mA and 37 mW at 28 V. The 10k
  ran at 75 % of its 0603 rating at 29.4 V.
* S6, bay node: F1 (CAM_5V) goes from the 0.5 A PTC to SMD1206P075TF
  (RUILON, C20987, new catalog key pptc750): 0.75 A hold, 1.5 A trip,
  the same 1206 footprint. It is extended like C20799, so no fee changes.
  - Arducam gives the Mega 317 mA working: with the LEDs that is
    ~0.42 A on CAM_5V, where the 0.5 A part holds ~0.31 A at 70 C.
  - The camera pod's LDO tab gets the copper its routing leaves: a
    top-side +3V3 pour round the tab and a bottom-side island, joined by
    three vias. U1 drops ~0.5 W at 317 mA. The routing is unchanged.
  - The "~120 mA" notes go to 317 mA (node and pod design.py,
    electronics.md).
  - The bay's worst case follows: <= 2.25 A on +5V, the buck's inductor
    peaking at ~2.65 A (under its 2.9 A minimum limit), 13.5 W from
    VRACK (power-distribution-review.md, the buck notes).

The routed PCBs keep their routing.
- Node and hub: only the changed parts' properties (KiCad's Python, as
  pcbgen sets them).
- Pod: the two new zones and three vias, refilled.
- ERC 0, DRC 0, unconnected 0, parity 0 on all three (run on the Mac:
  zephyrbox didn't answer).
- keep_unchanged kept the node's renders and the hub's Gerbers. The
  hub's bottom render is restored: 9 pixels of via-hole noise, as before.
- The pod's renders, Gerbers and viewer GLB chang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
Parts:
- R29: value 470k -> 150k; LCSC C23178 -> C22807; MPN 0603WAF4703T5E -> 0603WAF1503T5E
Changed lines of the file:
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@@
 			)
 		)
-		(property "Value" "470k"
+		(property "Value" "150k"
 			(at 93.016 114.3 0)
 			(effects
@@
 			)
 		)
-		(property "Description" "Resistor 470k 0603"
+		(property "Description" "Resistor 150k 0603"
 			(at 88.9 113.03 0)
 			(effects
@@
 			)
 		)
-		(property "LCSC" "C23178"
+		(property "LCSC" "C22807"
 			(at 88.9 113.03 0)
 			(effects
@@
 			)
 		)
-		(property "MPN" "0603WAF4703T5E"
+		(property "MPN" "0603WAF1503T5E"
 			(at 88.9 113.03 0)
 			(effects
@@
 		)
 	)
-	(text_box "CAN (docs/can.md): one bus for the rack, a star from the hub; both terminations sit in the hub.\n  250 kbit/s (125 kbit/s fallback).  TJA1462AT (SIC): VCC 5 V, VIO 3.3 V, bus pins −36/+40 V, passive unpowered.\nPOS: active-high 3.3 V token.  From reset the node holds POS_OUT low; when POS_IN goes high and it has\n  no address yet, it answers with its MAC, takes (row, position) from the hub, then raises POS_OUT.\n  R29 keeps POS_IN low with no cable; the next node's 470k keeps POS_OUT low before firmware."
+	(text_box "CAN (docs/can.md): one bus for the rack, a star from the hub; both terminations sit in the hub.\n  250 kbit/s (125 kbit/s fallback).  TJA1462AT (SIC): VCC 5 V, VIO 3.3 V, bus pins −36/+40 V, passive unpowered.\nPOS: active-high 3.3 V token.  From reset the node holds POS_OUT low; when POS_IN goes high and it has\n  no address yet, it answers with its MAC, takes (row, position) from the hub, then raises POS_OUT.\n  R29 keeps POS_IN low with no cable; the next node's 150k keeps POS_OUT low before firmware."
 		(exclude_from_sim no)
 		(at 15.24 177.8 0)
