File: electronics/bay-node/power.kicad_sch (KiCad schematic)
At the start: 23 parts, among them J1 ROW IN, J2 ROW OUT, Q1 SUD50P06-15, U1 LMR51635YDDCR, U2 AMS1117-3.3

Commit message: Bay node 74 × 90: no J4, AUX and DATA side entry on the right edge
The node grows 10 mm on the right and drops the DUT receptacle J4 (the
user's option B, 2026-10-19): every DUT hangs on the DATA lead.

- J7 (DATA, S8B) and J5 (AUX, S6B) are side entry on the right edge,
  facing the drag chain; J6 (CAM) stays vertical at the rear right, its
  lead straight back, east of the antenna keep-out.  J2 and the right
  holes (x 70.5) move to the new edge; the front half and the left holes
  stay (the tray's access holes, a09923f).
- U8 is the last part before J7; the hand-drawn HS chain ends on J7's
  pads (DUT_CONN matched with its two vias).  R14/R15 go with J4.
- +5V at 5.24 V (FB 100k/18k) for the DATA board at 1.4 A; INA226 Vbus
  on Vin- at its pins.
- Docs: electronics, cabling, assembly, power (no batteries on rack
  DUTs), the third Konnect round; BOM and JLC estimate (≈ $328), web
  scene's DATA plug, notice NODE_DATA.

Co-Authored-By: Claude Opus 5.5 <noreply@anthropic.com>
Parts:
- R4: value 120k -> 100k; LCSC C25808 -> C25803; MPN 0603WAF1203T5E -> 0603WAF1003T5E
- R5: value 22k -> 18k; LCSC C31850 -> C25810; MPN 0603WAF2202T5E -> 0603WAF1802T5E
Changed lines of the file:
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@@
 			)
 		)
-		(property "Value" "120k"
+		(property "Value" "100k"
 			(at 192.076 124.46 0)
 			(effects
@@
 			)
 		)
-		(property "Description" "Resistor 120k 0603"
+		(property "Description" "Resistor 100k 0603"
 			(at 187.96 123.19 0)
 			(effects
@@
 			)
 		)
-		(property "LCSC" "C25808"
+		(property "LCSC" "C25803"
 			(at 187.96 123.19 0)
 			(effects
@@
 			)
 		)
-		(property "MPN" "0603WAF1203T5E"
+		(property "MPN" "0603WAF1003T5E"
 			(at 187.96 123.19 0)
 			(effects
@@
 			)
 		)
-		(property "Value" "22k"
+		(property "Value" "18k"
 			(at 191.551 142.24 0)
 			(effects
@@
 			)
 		)
-		(property "Description" "Resistor 22k 0603"
+		(property "Description" "Resistor 18k 0603"
 			(at 187.96 140.97 0)
 			(effects
@@
 			)
 		)
-		(property "LCSC" "C31850"
+		(property "LCSC" "C25810"
 			(at 187.96 140.97 0)
 			(effects
@@
 			)
 		)
-		(property "MPN" "0603WAF2202T5E"
+		(property "MPN" "0603WAF1802T5E"
 			(at 187.96 140.97 0)
 			(effects
@@
 		)
 	)
-	(text_box "LMR51635YDDCR: 1.1 MHz, PFM at light load with spread spectrum.  Values from TI SLUSF64B table 8-2 (5 V, 1.1 MHz):\n  L 3.3 µH (FXL0630, 9.5 A sat);  COUT 3 × 22 µF/25 V (≥ 33 µF left after DC-bias derating);  CIN 2 × 10 µF/50 V + 100 nF;  CB 100 nF.\nFB 120k/22k: VOUT = 0.8 V × (1 + 120/22) = 5.16 V, which covers the DUT switch + shunt drop.\nEN 1M/100k: the buck starts above 13.5 V and stops below 10.8 V (VEN 1.226 V, 0.241 V hysteresis), so no node\n  draws its low-voltage inrush while the hub's eFuse is soft-starting the row.\nLayout: C4/C2/C3 straddle U1's VIN and GND pins on the top layer; CIN, U1 and COUT share one top-side GND island\n  with vias to the In1 plane; the FB divider sits at the FB pin, its +5V sense comes from COUT on another layer.\nInput: SUD50P06 P-FET (reverse polarity, Vgs clamped by the 12 V zener); SMBJ33A clamps hot-plug ringing below 54 V (U1: 63 V abs max).\nVRACK is 20 V, or 28 V (EPR), from the hub's USB-C PD supply: SMBJ33A stands off 33 V (28 V + 5 % = 29.4 V), the buck runs\n  4.3–60 V and starts above 13.5 V, the P-FET and the zener clamp are rated 60 V / 12 V.  At 20 V a row draws more current: ≤ 1.6 A."
+	(text_box "LMR51635YDDCR: 1.1 MHz, PFM at light load with spread spectrum.  Values from TI SLUSF64B table 8-2 (5 V, 1.1 MHz):\n  L 3.3 µH (FXL0630, 9.5 A sat);  COUT 3 × 22 µF/25 V (≥ 33 µF left after DC-bias derating);  CIN 2 × 10 µF/50 V + 100 nF;  CB 100 nF.\nFB 100k/18k: VOUT = 0.8 V × (1 + 100/18) = 5.24 V: ≈ 4.75 V still reaches the DATA board at 1.4 A over 50 cm\n  of PH lead (switch, shunt, one PH pin each way); everything on +5V takes it (TCAN1462V ≤ 5.5 V).\nEN 1M/100k: the buck starts above 13.5 V and stops below 10.8 V (VEN 1.226 V, 0.241 V hysteresis), so no node\n  draws its low-voltage inrush while the hub's eFuse is soft-starting the row.\nLayout: C4/C2/C3 straddle U1's VIN and GND pins on the top layer; CIN, U1 and COUT share one top-side GND island\n  with vias to the In1 plane; the FB divider sits at the FB pin, its +5V sense comes from COUT on another layer.\nInput: SUD50P06 P-FET (reverse polarity, Vgs clamped by the 12 V zener); SMBJ33A clamps hot-plug ringing below 54 V (U1: 63 V abs max).\nVRACK is 20 V, or 28 V (EPR), from the hub's USB-C PD supply: SMBJ33A stands off 33 V (28 V + 5 % = 29.4 V), the buck runs\n  4.3–60 V and starts above 13.5 V, the P-FET and the zener clamp are rated 60 V / 12 V.  At 20 V a row draws more current: ≤ 1.6 A."
 		(exclude_from_sim no)
 		(at 15.24 162.56 0)
-		(size 279.4 26.67)
+		(size 279.4 29.21)
 		(margins 1.5 1.5 1.5 1.5)
 		(stroke

Commit message: CAN transceiver: the TJA1462AT on the hub and the node
The TCAN1462V (C7399456) had no LCSC stock on 2026-10-18 and 19, and
JLC's quote of the hub asked for another part.  The user chose NXP's
TJA1462AT/0Z (C3234095, 10 500 in stock) for both boards (hub U6, node
U11): the same SOIC-8 pinout (VIO on pin 5, STB on pin 8), signal
improvement kept, bus pins -36/+40 V instead of ±58 V.  The TCAN1462V
and the TCAN1044AV stay the alternates.

Both boards regenerated and the same Freerouting sessions re-imported
(tracks and vias unchanged): ERC 0, DRC 0 errors (the hub's known C8
silkscreen warning), 0 unconnected, parity 0, JLC READY.  The CPL keeps
its 270° correction (C3234095 was already in build_board.py).

Docs: can.md, electronics.md, firmware comments and pin tables,
bom/sourcing.md, which also notes that JLC unticks the USB4105 (hard to
process, $0.03 a piece): tick it again at every order.

Co-Authored-By: Claude Opus 5.5 <noreply@anthropic.com>
Changed lines of the file:
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@@
 		)
 	)
-	(text_box "LMR51635YDDCR: 1.1 MHz, PFM at light load with spread spectrum.  Values from TI SLUSF64B table 8-2 (5 V, 1.1 MHz):\n  L 3.3 µH (FXL0630, 9.5 A sat);  COUT 3 × 22 µF/25 V (≥ 33 µF left after DC-bias derating);  CIN 2 × 10 µF/50 V + 100 nF;  CB 100 nF.\nFB 100k/18k: VOUT = 0.8 V × (1 + 100/18) = 5.24 V: ≈ 4.75 V still reaches the DATA board at 1.4 A over 50 cm\n  of PH lead (switch, shunt, one PH pin each way); everything on +5V takes it (TCAN1462V ≤ 5.5 V).\nEN 1M/100k: the buck starts above 13.5 V and stops below 10.8 V (VEN 1.226 V, 0.241 V hysteresis), so no node\n  draws its low-voltage inrush while the hub's eFuse is soft-starting the row.\nLayout: C4/C2/C3 straddle U1's VIN and GND pins on the top layer; CIN, U1 and COUT share one top-side GND island\n  with vias to the In1 plane; the FB divider sits at the FB pin, its +5V sense comes from COUT on another layer.\nInput: SUD50P06 P-FET (reverse polarity, Vgs clamped by the 12 V zener); SMBJ33A clamps hot-plug ringing below 54 V (U1: 63 V abs max).\nVRACK is 20 V, or 28 V (EPR), from the hub's USB-C PD supply: SMBJ33A stands off 33 V (28 V + 5 % = 29.4 V), the buck runs\n  4.3–60 V and starts above 13.5 V, the P-FET and the zener clamp are rated 60 V / 12 V.  At 20 V a row draws more current: ≤ 1.6 A."
+	(text_box "LMR51635YDDCR: 1.1 MHz, PFM at light load with spread spectrum.  Values from TI SLUSF64B table 8-2 (5 V, 1.1 MHz):\n  L 3.3 µH (FXL0630, 9.5 A sat);  COUT 3 × 22 µF/25 V (≥ 33 µF left after DC-bias derating);  CIN 2 × 10 µF/50 V + 100 nF;  CB 100 nF.\nFB 100k/18k: VOUT = 0.8 V × (1 + 100/18) = 5.24 V: ≈ 4.75 V still reaches the DATA board at 1.4 A over 50 cm\n  of PH lead (switch, shunt, one PH pin each way); everything on +5V takes it (TJA1462AT ≤ 5.5 V).\nEN 1M/100k: the buck starts above 13.5 V and stops below 10.8 V (VEN 1.226 V, 0.241 V hysteresis), so no node\n  draws its low-voltage inrush while the hub's eFuse is soft-starting the row.\nLayout: C4/C2/C3 straddle U1's VIN and GND pins on the top layer; CIN, U1 and COUT share one top-side GND island\n  with vias to the In1 plane; the FB divider sits at the FB pin, its +5V sense comes from COUT on another layer.\nInput: SUD50P06 P-FET (reverse polarity, Vgs clamped by the 12 V zener); SMBJ33A clamps hot-plug ringing below 54 V (U1: 63 V abs max).\nVRACK is 20 V, or 28 V (EPR), from the hub's USB-C PD supply: SMBJ33A stands off 33 V (28 V + 5 % = 29.4 V), the buck runs\n  4.3–60 V and starts above 13.5 V, the P-FET and the zener clamp are rated 60 V / 12 V.  At 20 V a row draws more current: ≤ 1.6 A."
 		(exclude_from_sim no)
 		(at 15.24 162.56 0)

Commit message: Hub 37 and node 38 part types: more values merged
From the JLC cost session's list (it does the analysis, this session
edits the boards).  No footprint or track moves; both boards regenerated
on their Freerouting sessions (node 996/386, hub 1241/593 segments/vias),
ERC 0, DRC 0 errors (the hub's known C8 silkscreen warning), parity 0.

- Hub: the IMON filters and the CAN split caps on the dVdT caps' 22 nF
  (IMON RC 22 µs; the split cap only filters common mode): 38 -> 37 types,
  -$17.05 of feeders against the quote, order ≈ $212.77.
- Node: buck EN 100k/10k (same 13.5 V / 10.8 V), PC_DET 10k/18k (3.2 V),
  I²C pull-ups 5.1k, AUX VREF 33 Ω: 42 -> 38 types, estimate ≈ $322.77.

Docs: electronics.md (the hub's types per block, the node's estimate),
can.md, firmware pin tables.

Co-Authored-By: Claude Opus 5.5 <noreply@anthropic.com>
Parts:
- R2: value 1M -> 100k; LCSC C22935 -> C25803; MPN 0603WAF1004T5E -> 0603WAF1003T5E
- R3: value 100k -> 10k; LCSC C25803 -> C25804; MPN 0603WAF1003T5E -> 0603WAF1002T5E
Changed lines of the file:
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@@
 			)
 		)
-		(property "Value" "1M"
-			(at 76.726 106.68 0)
+		(property "Value" "100k"
+			(at 77.776 106.68 0)
 			(effects
 				(font
@@
 			)
 		)
-		(property "Description" "Resistor 1M 0603"
+		(property "Description" "Resistor 100k 0603"
 			(at 73.66 105.41 0)
 			(effects
@@
 			)
 		)
-		(property "LCSC" "C22935"
+		(property "LCSC" "C25803"
 			(at 73.66 105.41 0)
 			(effects
@@
 			)
 		)
-		(property "MPN" "0603WAF1004T5E"
+		(property "MPN" "0603WAF1003T5E"
 			(at 73.66 105.41 0)
 			(effects
@@
 			)
 		)
-		(property "Value" "100k"
-			(at 77.776 124.46 0)
+		(property "Value" "10k"
+			(at 77.251 124.46 0)
 			(effects
 				(font
@@
 			)
 		)
-		(property "Description" "Resistor 100k 0603"
+		(property "Description" "Resistor 10k 0603"
 			(at 73.66 123.19 0)
 			(effects
@@
 			)
 		)
-		(property "LCSC" "C25803"
+		(property "LCSC" "C25804"
 			(at 73.66 123.19 0)
 			(effects
@@
 			)
 		)
-		(property "MPN" "0603WAF1003T5E"
+		(property "MPN" "0603WAF1002T5E"
 			(at 73.66 123.19 0)
 			(effects
@@
 		)
 	)
-	(text_box "LMR51635YDDCR: 1.1 MHz, PFM at light load with spread spectrum.  Values from TI SLUSF64B table 8-2 (5 V, 1.1 MHz):\n  L 3.3 µH (FXL0630, 9.5 A sat);  COUT 3 × 22 µF/25 V (≥ 33 µF left after DC-bias derating);  CIN 2 × 10 µF/50 V + 100 nF;  CB 100 nF.\nFB 100k/18k: VOUT = 0.8 V × (1 + 100/18) = 5.24 V: ≈ 4.75 V still reaches the DATA board at 1.4 A over 50 cm\n  of PH lead (switch, shunt, one PH pin each way); everything on +5V takes it (TJA1462AT ≤ 5.5 V).\nEN 1M/100k: the buck starts above 13.5 V and stops below 10.8 V (VEN 1.226 V, 0.241 V hysteresis), so no node\n  draws its low-voltage inrush while the hub's eFuse is soft-starting the row.\nLayout: C4/C2/C3 straddle U1's VIN and GND pins on the top layer; CIN, U1 and COUT share one top-side GND island\n  with vias to the In1 plane; the FB divider sits at the FB pin, its +5V sense comes from COUT on another layer.\nInput: SUD50P06 P-FET (reverse polarity, Vgs clamped by the 12 V zener); SMBJ33A clamps hot-plug ringing below 54 V (U1: 63 V abs max).\nVRACK is 20 V, or 28 V (EPR), from the hub's USB-C PD supply: SMBJ33A stands off 33 V (28 V + 5 % = 29.4 V), the buck runs\n  4.3–60 V and starts above 13.5 V, the P-FET and the zener clamp are rated 60 V / 12 V.  At 20 V a row draws more current: ≤ 1.6 A."
+	(text_box "LMR51635YDDCR: 1.1 MHz, PFM at light load with spread spectrum.  Values from TI SLUSF64B table 8-2 (5 V, 1.1 MHz):\n  L 3.3 µH (FXL0630, 9.5 A sat);  COUT 3 × 22 µF/25 V (≥ 33 µF left after DC-bias derating);  CIN 2 × 10 µF/50 V + 100 nF;  CB 100 nF.\nFB 100k/18k: VOUT = 0.8 V × (1 + 100/18) = 5.24 V: ≈ 4.75 V still reaches the DATA board at 1.4 A over 50 cm\n  of PH lead (switch, shunt, one PH pin each way); everything on +5V takes it (TJA1462AT ≤ 5.5 V).\nEN 100k/10k: the buck starts above 13.5 V and stops below 10.8 V (VEN 1.226 V, 0.241 V hysteresis), so no node\n  draws its low-voltage inrush while the hub's eFuse is soft-starting the row.\nLayout: C4/C2/C3 straddle U1's VIN and GND pins on the top layer; CIN, U1 and COUT share one top-side GND island\n  with vias to the In1 plane; the FB divider sits at the FB pin, its +5V sense comes from COUT on another layer.\nInput: SUD50P06 P-FET (reverse polarity, Vgs clamped by the 12 V zener); SMBJ33A clamps hot-plug ringing below 54 V (U1: 63 V abs max).\nVRACK is 20 V, or 28 V (EPR), from the hub's USB-C PD supply: SMBJ33A stands off 33 V (28 V + 5 % = 29.4 V), the buck runs\n  4.3–60 V and starts above 13.5 V, the P-FET and the zener clamp are rated 60 V / 12 V.  At 20 V a row draws more current: ≤ 1.6 A."
 		(exclude_from_sim no)
 		(at 15.24 162.56 0)

Commit message: PCBA review: hub and node fixes before the order
On main's CH224A hub and the bay node v0.5.

Power hub:
- CPL: the side LEDs (C598310, C4555382) +0.825 mm, their polarity
  proven from JLC's own footprints (and C495809 at 270 deg in the table,
  for the IRF7842 the AP33772S hub had).
- Rows: SHDN pull-downs 10k, so rows stay off without firmware (100k
  gave 1 V at the pin's 10 uA); a B5819W at each row output for the
  cable's kick; the red FAULT LEDs fed from their ROW_EN, so a row that
  is simply off shows no fault.
- In2's VRACK band 8 mm wide; the console's USB pair hand-routed on
  F.Cu over In1 (U5's channels in the pair's order), EN's capacitor at
  the module's pin; reliefs on both pads of C2, C10, R3, C11-C14; notes
  corrected, the outputs sheet on A2.
- The PESD2CAN kept and documented (no stocked CAN TVS stays off at
  29.4 V and clamps under +40 V).

Bay node:
- SW3 placed on its pegs (-0.55 mm, Shouhan's land pattern); 2.2k I2C
  pull-ups; POS_IN 470k; AUX_VREF 1k; 100k on SVC; U9's input on a +5V
  island with three vias, C20 at its pins; C12 relieved; the camera note
  and the catalog's MPN text corrected.

Both re-routed: ERC 0, DRC 0 (the known C8 silkscreen warning), parity
0; CPL audit against JLC's footprints: every part agrees but SW3's pads
(0.13 mm, on purpose).  Bring-up measurements in assembly.md, the
resolution in pcba-review.md.

Co-Authored-By: Claude Opus 5.5 <noreply@anthropic.com>
Parts:
- Q1: value SUD50P06-15 -> SUD50P06-15(UMW); MPN SUD50P06-15 -> SUD50P06-15(UMW); Manufacturer UMW / Vishay -> UMW
Changed lines of the file:
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@@
 			)
 		)
-		(property "Value" "SUD50P06-15"
-			(at 75.625 25.908 90)
+		(property "Value" "SUD50P06-15(UMW)"
+			(at 78.25 25.908 90)
 			(effects
 				(font
@@
 			)
 		)
-		(property "MPN" "SUD50P06-15"
+		(property "MPN" "SUD50P06-15(UMW)"
 			(at 60.96 33.02 0)
 			(effects
@@
 			)
 		)
-		(property "Manufacturer" "UMW / Vishay"
+		(property "Manufacturer" "UMW"
 			(at 60.96 33.02 0)
 			(effects
