File: electronics/bay-node/usb.kicad_sch (KiCad schematic)
At the start: 20 parts, among them J3 PC, J7 DATA, SW3 SERVICE, U4 USBLC6-2SC6, U5 MUX_PC, U6 MUX_DUT, U7 SN74LVC1G32DBVR, U8 USBLC6-2SC6

Commit message: PCBA review: hub and node fixes before the order
On main's CH224A hub and the bay node v0.5.

Power hub:
- CPL: the side LEDs (C598310, C4555382) +0.825 mm, their polarity
  proven from JLC's own footprints (and C495809 at 270 deg in the table,
  for the IRF7842 the AP33772S hub had).
- Rows: SHDN pull-downs 10k, so rows stay off without firmware (100k
  gave 1 V at the pin's 10 uA); a B5819W at each row output for the
  cable's kick; the red FAULT LEDs fed from their ROW_EN, so a row that
  is simply off shows no fault.
- In2's VRACK band 8 mm wide; the console's USB pair hand-routed on
  F.Cu over In1 (U5's channels in the pair's order), EN's capacitor at
  the module's pin; reliefs on both pads of C2, C10, R3, C11-C14; notes
  corrected, the outputs sheet on A2.
- The PESD2CAN kept and documented (no stocked CAN TVS stays off at
  29.4 V and clamps under +40 V).

Bay node:
- SW3 placed on its pegs (-0.55 mm, Shouhan's land pattern); 2.2k I2C
  pull-ups; POS_IN 470k; AUX_VREF 1k; 100k on SVC; U9's input on a +5V
  island with three vias, C20 at its pins; C12 relieved; the camera note
  and the catalog's MPN text corrected.

Both re-routed: ERC 0, DRC 0 (the known C8 silkscreen warning), parity
0; CPL audit against JLC's footprints: every part agrees but SW3's pads
(0.13 mm, on purpose).  Bring-up measurements in assembly.md, the
resolution in pcba-review.md.

Co-Authored-By: Claude Opus 5.5 <noreply@anthropic.com>
Parts:
- added R39: 100k, Resistor_SMD:R_0603_1608Metric, symbol Device:R
Connections:
- net GND: now also R39.2
- net SVC: now also R39.1
Changed lines of the file:
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@@
+		)
+	)
+	(symbol
+		(lib_id "Device:R")
+		(at 198.12 203.2 0)
+		(unit 1)
+		(exclude_from_sim no)
+		(in_bom yes)
+		(on_board yes)
+		(dnp no)
+		(fields_autoplaced yes)
+		(property "Reference" "R39"
+			(at 201.711 201.93 0)
+			(effects
+				(font
+					(size 1.27 1.27)
+				)
+			)
+		)
+		(property "Value" "100k"
+			(at 202.236 204.47 0)
+			(effects
+				(font
+					(size 1.27 1.27)
+				)
+			)
+		)
+		(property "Footprint" "Resistor_SMD:R_0603_1608Metric"
+			(at 198.12 203.2 0)
+			(effects
+				(font
+					(size 1.27 1.27)
+				)
+				(hide yes)
+			)
+		)
+		(property "Datasheet" ""
+			(at 198.12 203.2 0)
+			(effects
+				(font
+					(size 1.27 1.27)
+				)
+				(hide yes)
+			)
+		)
+		(property "Description" "Resistor 100k 0603"
+			(at 198.12 203.2 0)
+			(effects
+				(font
+					(size 1.27 1.27)
+				)
+				(hide yes)
+			)
+		)
+		(property "LCSC" "C25803"
+			(at 198.12 203.2 0)
+			(effects
+				(font
+					(size 1.27 1.27)
+				)
+				(hide yes)
+			)
+		)
+		(property "MPN" "0603WAF1003T5E"
+			(at 198.12 203.2 0)
+			(effects
+				(font
+					(size 1.27 1.27)
+				)
+				(hide yes)
+			)
+		)
+		(property "Manufacturer" "UNI-ROYAL(Uniroyal Elec)"
+			(at 198.12 203.2 0)
+			(effects
+				(font
+					(size 1.27 1.27)
+				)
+				(hide yes)
+			)
+		)
+		(pin "1"
+		)
+		(pin "2"
+		)
+		(instances
+			(project "bay-node"
+				(path "/76847c0c-2f76-566c-8109-428b2bf58b3f/c87ef098-13d8-5d4c-814e-a4c6487f5259"
+					(reference "R39")
+					(unit 1)
+				)
+			)
+		)
+	)
+	(wire
+		(pts
+			(xy 198.12 199.39)
+			(xy 198.12 196.85)
+		)
+		(stroke
+			(width 0)
+			(type default)
+		)
+	)
+	(global_label "SVC"
+		(shape bidirectional)
+		(at 198.12 196.85 90)
+		(fields_autoplaced yes)
+		(effects
+			(font
+				(size 1.27 1.27)
+			)
+			(justify left)
+		)
+		(property "Intersheetrefs" "${INTERSHEET_REFS}"
+			(at 198.12 196.85 0)
+			(effects
+				(font
+					(size 1.27 1.27)
+				)
+				(justify left)
+				(hide yes)
+			)
+		)
+	)
+	(wire
+		(pts
+			(xy 198.12 207.01)
+			(xy 198.12 209.55)
+		)
+		(stroke
+			(width 0)
+			(type default)
+		)
+	)
+	(symbol
+		(lib_id "power:GND")
+		(at 198.12 209.55 0)
+		(unit 1)
+		(exclude_from_sim no)
+		(in_bom yes)
+		(on_board yes)
+		(dnp no)
+		(fields_autoplaced yes)
+		(property "Reference" "#PWR04021"
+			(at 198.12 209.55 0)
+			(effects
+				(font
+					(size 1.27 1.27)
+				)
+				(hide yes)
+			)
+		)
+		(property "Value" "GND"
+			(at 198.12 213.36 0)
+			(effects
+				(font
+					(size 1.27 1.27)
+				)
+			)
+		)
+		(property "Footprint" ""
+			(at 198.12 209.55 0)
+			(effects
+				(font
+					(size 1.27 1.27)
+				)
+				(hide yes)
+			)
+		)
+		(property "Datasheet" ""
+			(at 198.12 209.55 0)
+			(effects
+				(font
+					(size 1.27 1.27)
+				)
+				(hide yes)
+			)
+		)
+		(property "Description" ""
+			(at 198.12 209.55 0)
+			(effects
+				(font
+					(size 1.27 1.27)
+				)
+				(hide yes)
+			)
+		)
+		(pin "1"
+		)
+		(instances
+			(project "bay-node"
+				(path "/76847c0c-2f76-566c-8109-428b2bf58b3f/c87ef098-13d8-5d4c-814e-a4c6487f5259"
+					(reference "#PWR04021")
+					(unit 1)
+				)
+			)
 		)
 	)
@@
 		(dnp no)
 		(fields_autoplaced yes)
-		(property "Reference" "#PWR04021"
+		(property "Reference" "#PWR04022"
 			(at 71.12 121.92 0)
 			(effects
@@
 			(project "bay-node"
 				(path "/76847c0c-2f76-566c-8109-428b2bf58b3f/c87ef098-13d8-5d4c-814e-a4c6487f5259"
-					(reference "#PWR04021")
+					(reference "#PWR04022")
 					(unit 1)
 				)
@@
 		(dnp no)
 		(fields_autoplaced yes)
-		(property "Reference" "#PWR04022"
+		(property "Reference" "#PWR04023"
 			(at 193.04 40.64 0)
 			(effects
@@
 			(project "bay-node"
 				(path "/76847c0c-2f76-566c-8109-428b2bf58b3f/c87ef098-13d8-5d4c-814e-a4c6487f5259"
-					(reference "#PWR04022")
+					(reference "#PWR04023")
 					(unit 1)
 				)
@@
 		(dnp no)
 		(fields_autoplaced yes)
-		(property "Reference" "#PWR04023"
+		(property "Reference" "#PWR04024"
 			(at 264.16 40.64 0)
 			(effects
@@
 			(project "bay-node"
 				(path "/76847c0c-2f76-566c-8109-428b2bf58b3f/c87ef098-13d8-5d4c-814e-a4c6487f5259"
-					(reference "#PWR04023")
+					(reference "#PWR04024")
 					(unit 1)
 				)
@@
 		(dnp no)
 		(fields_autoplaced yes)
-		(property "Reference" "#PWR04024"
+		(property "Reference" "#PWR04025"
 			(at 363.22 213.36 0)
 			(effects
@@
 			(project "bay-node"
 				(path "/76847c0c-2f76-566c-8109-428b2bf58b3f/c87ef098-13d8-5d4c-814e-a4c6487f5259"
-					(reference "#PWR04024")
+					(reference "#PWR04025")
 					(unit 1)
 				)
@@
 		(dnp no)
 		(fields_autoplaced yes)
-		(property "Reference" "#PWR04025"
+		(property "Reference" "#PWR04026"
 			(at 363.22 220.98 0)
 			(effects
@@
 			(project "bay-node"
 				(path "/76847c0c-2f76-566c-8109-428b2bf58b3f/c87ef098-13d8-5d4c-814e-a4c6487f5259"
-					(reference "#PWR04025")
+					(reference "#PWR04026")
 					(unit 1)
 				)
@@
 		(dnp no)
 		(fields_autoplaced yes)
-		(property "Reference" "#PWR04026"
+		(property "Reference" "#PWR04027"
 			(at 101.6 167.64 0)
 			(effects
@@
 			(project "bay-node"
 				(path "/76847c0c-2f76-566c-8109-428b2bf58b3f/c87ef098-13d8-5d4c-814e-a4c6487f5259"
-					(reference "#PWR04026")
+					(reference "#PWR04027")
 					(unit 1)
 				)
@@
 		(dnp no)
 		(fields_autoplaced yes)
-		(property "Reference" "#PWR04027"
+		(property "Reference" "#PWR04028"
 			(at 167.64 180.34 0)
 			(effects
@@
 			(project "bay-node"
 				(path "/76847c0c-2f76-566c-8109-428b2bf58b3f/c87ef098-13d8-5d4c-814e-a4c6487f5259"
-					(reference "#PWR04027")
+					(reference "#PWR04028")
 					(unit 1)
 				)
@@
 		(dnp no)
 		(fields_autoplaced yes)
-		(property "Reference" "#PWR04028"
+		(property "Reference" "#PWR04029"
 			(at 167.64 195.58 0)
 			(effects
@@
 			(project "bay-node"
 				(path "/76847c0c-2f76-566c-8109-428b2bf58b3f/c87ef098-13d8-5d4c-814e-a4c6487f5259"
-					(reference "#PWR04028")
+					(reference "#PWR04029")
 					(unit 1)
 				)

Commit message: Datasheet audit F1-F6: the pod's AP2114H, STB 5.1k, PC_DET hysteresis, the camera ESD's 100 nF, the eFuse step
The user approved the audit's fixes for the node, the hub and the pod
("Go pour 1"); docs/datasheet-audit.md marks F1-F6 applied.

* F1, camera pod: U1 AMS1117-3.3 -> AP2114H-3.3TRG1 (C150716, catalog
  ldo_1a, the node's U2).
  - The AMS1117 is specified stable only with 22 uF tantalum; the
    AP2114H is stable with the ceramic C2.
  - Same SOT-223 pinout, copper (the +3V3 pour and island round the
    tab stay) and 180 deg CPL correction.
  - One more extended type on the pod's Economic order: +$3.09 and
    $0.05 of parts (JLC_SINCE_QUOTE).
* F2, power hub: R214 (TJA1462 STB pull-down) 10k -> 5.1k (C23186,
  already on the board). With IO9 floating, STB's internal pull-up
  (20 kOhm minimum) left it at up to 1.10 V, over VIL 0.99 V.
* F3, bay node: R42 150k from MUX_SEL back to PC_DET, beside U7 (C22807,
  on the board since S1).
  - The laptop's VBUS rises at ~50 us/V through R11/R12, where the
    LVC1G32 wants <= 10 ns/V and warns of oscillation.
  - This gives ~0.14 V of hysteresis.
* F4, bay node: C28 100 nF (C14663) on U12/U13's VBUS pins (+3V3), above
  U12 by its pin 5. Between the two ICs their courtyards leave no room.
* F5, node and hub: firmware.md's first-flash procedure gains the
  irreversible DIS_USB_OTG_DOWNLOAD_MODE eFuse step. In USB-OTG
  download boot the ROM drives IO40 high: the node's DUT_FLT_N, the
  hub's PD_SCL. Nothing is burnt.
* F6, notes, hub:
  - the IMON filter is 0.9 ms, not 47 us: the pin is a current source;
  - the buck stops at ~3.8 V (internal UVLO);
  - SHDN turns on at >= 1 V;
  - the soft start stays under the limit only typically;
  - the CH224A note follows CH224 V2.1: the source PDOs are listed for
    both parts and readable under 100 W, which is still to check with
    ours (review R3); single-byte transfers; no "same die".
* F6, notes, node: TPS2553D; the LDO's 1.94 V x 0.4 A ~ 0.8 W; L1's
  7.5 A guarante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
Parts:
- added R42: 150k, Resistor_SMD:R_0603_1608Metric, symbol Device:R
Connections:
- net MUX_SEL: now also R42.1
- net PC_DET: now also R42.2
Changed lines of the file:
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@@
 		(comment 1 "ESP32-S3 USB/IP host for one bay of the hw-testing-rack shelf")
 		(comment 2 "Generated from electronics/bay-node/design.py — edit the Python, then regenerate")
-		(comment 3 "Row bus 20–28 V + CAN + POS in/out · 5 V/1.4 A switched DUT port · USB 2.0 muxes · INA226 · AUX")
+		(comment 3 "Row bus 20–28 V + CAN + POS in/out · 5 V/1.4 A switched DUT power on the DATA lead · USB 2.0 muxes · INA226 · AUX")
 	)
 	(symbol
@@
 			)
 		)
+	)
+	(symbol
+		(lib_id "Device:R")
+		(at 152.4 208.28 0)
+		(unit 1)
+		(exclude_from_sim no)
+		(in_bom yes)
+		(on_board yes)
+		(dnp no)
+		(fields_autoplaced yes)
+		(property "Reference" "R42"
+			(at 155.991 207.01 0)
+			(effects
+				(font
+					(size 1.27 1.27)
+				)
+			)
+		)
+		(property "Value" "150k"
+			(at 156.516 209.55 0)
+			(effects
+				(font
+					(size 1.27 1.27)
+				)
+			)
+		)
+		(property "Footprint" "Resistor_SMD:R_0603_1608Metric"
+			(at 152.4 208.28 0)
+			(effects
+				(font
+					(size 1.27 1.27)
+				)
+				(hide yes)
+			)
+		)
+		(property "Datasheet" ""
+			(at 152.4 208.28 0)
+			(effects
+				(font
+					(size 1.27 1.27)
+				)
+				(hide yes)
+			)
+		)
+		(property "Description" "Resistor 150k 0603"
+			(at 152.4 208.28 0)
+			(effects
+				(font
+					(size 1.27 1.27)
+				)
+				(hide yes)
+			)
+		)
+		(property "LCSC" "C22807"
+			(at 152.4 208.28 0)
+			(effects
+				(font
+					(size 1.27 1.27)
+				)
+				(hide yes)
+			)
+		)
+		(property "MPN" "0603WAF1503T5E"
+			(at 152.4 208.28 0)
+			(effects
+				(font
+					(size 1.27 1.27)
+				)
+				(hide yes)
+			)
+		)
+		(property "Manufacturer" "UNI-ROYAL(Uniroyal Elec)"
+			(at 152.4 208.28 0)
+			(effects
+				(font
+					(size 1.27 1.27)
+				)
+				(hide yes)
+			)
+		)
+		(pin "1"
+		)
+		(pin "2"
+		)
+		(instances
+			(project "bay-node"
+				(path "/76847c0c-2f76-566c-8109-428b2bf58b3f/c87ef098-13d8-5d4c-814e-a4c6487f5259"
+					(reference "R42")
+					(unit 1)
+				)
+			)
+		)
+	)
+	(wire
+		(pts
+			(xy 152.4 204.47)
+			(xy 152.4 201.93)
+		)
+		(stroke
+			(width 0)
+			(type default)
+		)
+	)
+	(label "MUX_SEL"
+		(at 152.4 201.93 90)
+		(fields_autoplaced yes)
+		(effects
+			(font
+				(size 1.27 1.27)
+			)
+			(justify left bottom)
+		)
+	)
+	(wire
+		(pts
+			(xy 152.4 212.09)
+			(xy 152.4 214.63)
+		)
+		(stroke
+			(width 0)
+			(type default)
+		)
+	)
+	(global_label "PC_DET"
+		(shape bidirectional)
+		(at 152.4 214.63 270)
+		(fields_autoplaced yes)
+		(effects
+			(font
+				(size 1.27 1.27)
+			)
+			(justify right)
+		)
+		(property "Intersheetrefs" "${INTERSHEET_REFS}"
+			(at 152.4 214.63 0)
+			(effects
+				(font
+					(size 1.27 1.27)
+				)
+				(justify right)
+				(hide yes)
+			)
+		)
