File: electronics/bay-node/cam.kicad_sch (KiCad schematic)
At the start: 20 parts, among them J6 CAM, Q4 AO3400A, U12 USBLC6-2SC6, U13 USBLC6-2SC6

Commit message: Bay node: the camera SPI through its ESD, flow-through (BN-3)
A new finding of the flow-through check (electronics/tools/flowthru.py).
Each camera SPI line had U12/U13's two pins (1/6, 3/4) on one net,
bridged under the part, and the routes passed three of the four lines
by:
- SCK went from J6 to R31 round a detour, with both of U12's pins on
  stubs;
- MOSI left J6's side for R32 on B.Cu without crossing U12;
- MISO's U13.6 joined the R33 side through a loop, leaving U13.1 on a
  stub.
Only CS ran through.

The ESDs now carry two nets per line, as U4 and U8 do: CAM_*_C from J6
to the pin facing it (6 or 4), CAM_*_P from the other pin (1 or 3) to
the 33 ohm resistor.  No route can pass the part by any more.  The
eight nets were re-routed incrementally; every other track and via is
main's.  The stitching adds one GND via under U12, between its rows,
in the pour that the old MOSI bridge left free.  TP19-TP21 (MOSI, MISO,
CS) stay where they are, now on the _P side; TP18 (SCK) stays on the
lead side.

This supersedes the PCBA review's N6 (2026-10-19).  N6 accepted U12/U13
as a clamp beside the line at 4 MHz; the user has since approved making
every ESD flow-through (X2-1, Fabio's rule).  The datasheet audit's
"6-7 mm from J6, OK" only measured the distance, and is corrected along
with the Konnect review's note.

pcbgen.stitch_gnd no longer takes a GND pad that holds a via for
lonely.  TP22 got a pointless 0.3 mm track inside its own pad.

ERC 0, DRC 0, unconnected 0, parity 0.

Co-Authored-By: Claude Opus 5.5 <noreply@anthropic.com>
Parts:
- TP19: value CAM_MOSI_C -> CAM_MOSI_P
- TP20: value CAM_MISO_C -> CAM_MISO_P
- TP21: value CAM_CS_C -> CAM_CS_P
Connections:
- net CAM_CS_C: no longer R34.2, TP21.1, U13.3 (I/O2)
- net CAM_MISO_C: no longer R33.1, TP20.1, U13.1 (I/O1)
- net CAM_MOSI_C: no longer R32.2, TP19.1, U12.3 (I/O2)
- net CAM_SCK_C: no longer R31.2, U12.1 (I/O1)
- new net CAM_CS_P: R34.2, TP21.1, U13.3 (I/O2)
- new net CAM_MISO_P: R33.1, TP20.1, U13.1 (I/O1)
- new net CAM_MOSI_P: R32.2, TP19.1, U12.3 (I/O2)
- new net CAM_SCK_P: R31.2, U12.1 (I/O1)
Changed lines of the file:
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@@
 		)
 	)
-	(label "CAM_SCK_C"
+	(label "CAM_SCK_P"
 		(at 133.35 60.96 0)
 		(fields_autoplaced yes)
@@
 		)
 	)
-	(label "CAM_MOSI_C"
+	(label "CAM_MOSI_P"
 		(at 133.35 76.2 0)
 		(fields_autoplaced yes)
@@
 		)
 	)
-	(label "CAM_MISO_C"
+	(label "CAM_MISO_P"
 		(at 120.65 91.44 180)
 		(fields_autoplaced yes)
@@
 		)
 	)
-	(label "CAM_CS_C"
+	(label "CAM_CS_P"
 		(at 133.35 106.68 0)
 		(fields_autoplaced yes)
@@
 		)
 	)
-	(label "CAM_SCK_C"
+	(label "CAM_SCK_P"
 		(at 185.42 55.88 180)
 		(fields_autoplaced yes)
@@
 		)
 	)
-	(label "CAM_MOSI_C"
+	(label "CAM_MOSI_P"
 		(at 185.42 58.42 180)
 		(fields_autoplaced yes)
@@
 		)
 	)
-	(label "CAM_MISO_C"
+	(label "CAM_MISO_P"
 		(at 185.42 96.52 180)
 		(fields_autoplaced yes)
@@
 		)
 	)
-	(label "CAM_CS_C"
+	(label "CAM_CS_P"
 		(at 185.42 99.06 180)
 		(fields_autoplaced yes)
@@
 			)
 		)
-		(property "Value" "CAM_MOSI_C"
+		(property "Value" "CAM_MOSI_P"
 			(at 332.586 82.55 90)
 			(effects
@@
 		)
 	)
-	(label "CAM_MOSI_C"
+	(label "CAM_MOSI_P"
 		(at 345.44 81.28 0)
 		(fields_autoplaced yes)
@@
 			)
 		)
-		(property "Value" "CAM_MISO_C"
+		(property "Value" "CAM_MISO_P"
 			(at 350.366 82.55 90)
 			(effects
@@
 		)
 	)
-	(label "CAM_MISO_C"
+	(label "CAM_MISO_P"
 		(at 363.22 81.28 0)
 		(fields_autoplaced yes)
@@
 			)
 		)
-		(property "Value" "CAM_CS_C"
+		(property "Value" "CAM_CS_P"
 			(at 369.196 82.55 90)
 			(effects
@@
 		)
 	)
-	(label "CAM_CS_C"
+	(label "CAM_CS_P"
 		(at 381 81.28 0)
 		(fields_autoplaced yes)
