File: electronics/data-port-x6/port2.kicad_sch (KiCad schematic)
At the start: 34 parts, among them J201 PORT2, J202 PINS2, U201 TPS2553DBVR-1, U202 INA226AIDGSR, U203 USBLC6-2SC6, U205 H5VU25UC, U206 H5VU25UC, U207 LSF0108RKSR, U208 H5VU25UC, U209 H5VU25UC

Commit message: DATA x6: placement, the functions grouped as the study drew them
The board placed, not routed (DRC: only the unrouted links; ERC 0).  Bands, top to bottom:
- the co-processor (the v2's block, 31.1 mm west) and its SWD header under it; the six
  colour blocks (z 65-81); the hub (the v2's block, a row lower) with converter B
  (+5V_B, the top-right corner) over it;
- per port its pin chain right under its block (the H5VU25UC, the 100 ohm arrays, the
  LSF0108, two rows of 0402);
- converter A (+5V_A) west, the three crosspoints with a TCA9535 between two, J1 east with
  the lead's ESD and the I2C isolation beside it; the matrix expander (TCA9534A) and the
  -5 V inverter under the SWD header, by the co-processor;
- a corridor for the USB pairs, then each port's switch and current sense, then its VBUS
  22 uF, CC resistors and LED over the receptacle, the USBLC6 in the gap west of it (port
  1's over its receptacle: the cradle's band beside it).
- VIN's 33 uF and J3 (rear face) under the blocks' legend; the 3.3 V LDO under converter A.

The hub's south face DN1-5 now feeds USB-C 2-6 and its west face DN6 USB-C 1, so the pairs
come down and turn west in lanes, the lowest dropping off first, none crossing (DN7: the
co-processor).  The power plane: +3V3 over the clusters' split (y 64.6), +5V_A / +5V_B
under it either side of x 50, each fed from its converter down the cradle's band at its
end; no B.Cu track crosses the main splits.  Rear-face test points spaced so their names
do not overlap; each port number over its block.

Co-Authored-By: Claude Opus 5.5 <noreply@anthropic.com>
Changed lines of the file:
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@@
 		)
 	)
-	(text_box "Port 2 = hub port 2, busid 1-1.2; supplied by +5V_A.\nINA226 at 0x43; expander U2 (TCA9535, 0x20).\nILIM 47k: 0.50–0.62 A; the -1 latches off after 7.5 ms in limit, FAULT_N flags it.\nINA226 Vbus on the shunt's load-side sense pad (= VBUS).\nEN pulled down: the port stays off until the node switches it on.\nPins: P1–P8 → crosspoint X lines (as the DATA ×4 v2's map, a third chip for ports 5–6);\n  an unwired VREF stays ≈ 0.4 V, under the LSF0108's 0.65 V: the firmware keeps the port's\n  crosspoint switches open while its VREF reads under 0.65 V.\nESD: VREF through U208, RESET_N / BOOT_N through U209 (flow-through).\nVREF: the board's I/O supply, 0.95–3.6 V; a 5 V board with TTL inputs: its own 3.3 V pin.\nSource only (Rp from the switched VBUS); a back-feeding source trips the TPS2553 (latched).\nThe DUT's RESET/BOOT pull-ups ≥ 4.7k: against 1k, the 1k in series stops at ≈ 1.65 V.\nHeader: yellow; left column VREF 1 2 3 4 BOOT, right GND 5 6 7 8 RESET."
+	(text_box "Port 2 = hub port 1, busid 1-1.1; supplied by +5V_A.\nINA226 at 0x43; expander U2 (TCA9535, 0x20).\nILIM 47k: 0.50–0.62 A; the -1 latches off after 7.5 ms in limit, FAULT_N flags it.\nINA226 Vbus on the shunt's load-side sense pad (= VBUS).\nEN pulled down: the port stays off until the node switches it on.\nPins: P1–P8 → crosspoint X lines (as the DATA ×4 v2's map, a third chip for ports 5–6);\n  an unwired VREF stays ≈ 0.4 V, under the LSF0108's 0.65 V: the firmware keeps the port's\n  crosspoint switches open while its VREF reads under 0.65 V.\nESD: VREF through U208, RESET_N / BOOT_N through U209 (flow-through).\nVREF: the board's I/O supply, 0.95–3.6 V; a 5 V board with TTL inputs: its own 3.3 V pin.\nSource only (Rp from the switched VBUS); a back-feeding source trips the TPS2553 (latched).\nThe DUT's RESET/BOOT pull-ups ≥ 4.7k: against 1k, the 1k in series stops at ≈ 1.65 V.\nHeader: yellow; left column VREF 1 2 3 4 BOOT, right GND 5 6 7 8 RESET."
 		(exclude_from_sim no)
 		(at 284.48 157.48 0)
